Commit message: tweak kinect setup

File: costar_simulation/robot/kinect.xacro (robot description, xacro)
@@ -3,5 +3,5 @@
   <xacro:include filename="$(find costar_simulation)/robot/kinect_gazebo2.urdf.xacro"/>
   <xacro:include filename="$(find costar_simulation)/robot/kinect_properties2.xacro"/>
-  <xacro:property name="kinect_cam_py" value="0"/>
+  <xacro:property name="kinect_cam_py" value="1"/>
   <!-- Parameterised in part by the values in turtlebot_properties.urdf.xacro -->
   <xacro:macro name="sensor_kinect" params="parent">

File: costar_simulation/robot/kinect_properties2.xacro (robot description, xacro)
@@ -56,5 +56,5 @@
   </xacro:property>
 	<property name="pi" value="3.14159265" />
-	<property name="cam_px" value="-2" />
+	<property name="cam_px" value="0" />
 <!--	<property name="cam_py" value="-0.0125" /> Y varies for different configurations. get sets in sensors_urdf -->
 	<property name="cam_pz" value="1" />

File: costar_simulation/robot/ur5_joint_limited.xacro (robot description, xacro)
@@ -10,7 +10,7 @@
   <xacro:include filename="$(find ur5_robotiq_parallel_description)/urdf/robotiq_85/gripper.transmission.xacro" />
   <!-- Kinect -->
-  <xacro:include filename="$(find ur5_robotiq_parallel_description)/urdf/kinect/kinect.xacro"/>
-  <xacro:include filename="$(find ur5_robotiq_parallel_description)/urdf/kinect/kinect_properties2.xacro"/>
-  <xacro:include filename="$(find ur5_robotiq_parallel_description)/urdf/kinect/kinect_gazebo2.urdf.xacro"/>
+  <xacro:include filename="$(find costar_simulation)/robot/kinect.xacro"/>
+  <xacro:include filename="$(find costar_simulation)/robot/kinect_properties2.xacro"/>
+  <xacro:include filename="$(find costar_simulation)/robot/kinect_gazebo2.urdf.xacro"/>
   <property name="M_PI" value="3.14159"/>
   <!-- property list -->

Commit message: moving things around to make sure startup works properly

File: costar_simulation/robot/kinect.xacro (robot description, xacro)
@@ -3,5 +3,5 @@
   <xacro:include filename="$(find costar_simulation)/robot/kinect_gazebo2.urdf.xacro"/>
   <xacro:include filename="$(find costar_simulation)/robot/kinect_properties2.xacro"/>
-  <xacro:property name="kinect_cam_py" value="1"/>
+  <xacro:property name="kinect_cam_py" value="3"/>
   <!-- Parameterised in part by the values in turtlebot_properties.urdf.xacro -->
   <xacro:macro name="sensor_kinect" params="parent">
@@ -48,5 +48,6 @@
          (Hence, don't publish them additionally!) -->
 	<joint name="camera_depth_joint" type="fixed">
-	  <origin xyz="0 ${2 * -kinect_cam_py} 0" rpy="0 0 0" />
+    <!--<origin xyz="0 ${2 * -kinect_cam_py} 0" rpy="0 0 0" />-->
+	  <origin xyz="0 0 0" rpy="0 0 0" />
 	  <parent link="camera_rgb_frame" />
 	  <child link="camera_depth_frame" />

Commit message: setting up kinect sensor and robot

File: costar_simulation/robot/kinect.xacro (robot description, xacro)
@@ -3,9 +3,15 @@
   <xacro:include filename="$(find costar_simulation)/robot/kinect_gazebo2.urdf.xacro"/>
   <xacro:include filename="$(find costar_simulation)/robot/kinect_properties2.xacro"/>
-  <xacro:property name="kinect_cam_py" value="3"/>
+	<property name="pi" value="3.14159265" />
+	<property name="cam_px" value="1.0" />
+  <property name="cam_py" value="1.0"/>
+	<property name="cam_pz" value="1.0" />
+  <property name="cam_or" value="0.0" />
+	<property name="cam_op" value="${pi*0.25}" />
+	<property name="cam_oy" value="${pi*-0.5}" />
   <!-- Parameterised in part by the values in turtlebot_properties.urdf.xacro -->
   <xacro:macro name="sensor_kinect" params="parent">
     <joint name="camera_rgb_joint" type="fixed">
-      <origin xyz="${cam_px} ${kinect_cam_py} ${cam_pz}" rpy="${cam_or} ${cam_op} ${cam_oy}"/>
+      <origin xyz="${cam_px} ${cam_py} ${cam_pz}" rpy="${cam_or} ${cam_op} ${cam_oy}"/>
       <parent link="${parent}"/>
       <child link="camera_rgb_frame" />
@@ -19,5 +25,5 @@
     <link name="camera_rgb_optical_frame"/>
     <joint name="camera_joint" type="fixed">
-      <origin xyz="-0.031 ${-kinect_cam_py} -0.016" rpy="0 0 0"/>
+      <origin xyz="-0.031 ${-cam_py} -0.016" rpy="0 0 0"/>
       <parent link="camera_rgb_frame"/>
       <child link="camera_link"/>
@@ -48,5 +54,5 @@
          (Hence, don't publish them additionally!) -->
 	<joint name="camera_depth_joint" type="fixed">
-    <!--<origin xyz="0 ${2 * -kinect_cam_py} 0" rpy="0 0 0" />-->
+    <!--<origin xyz="0 ${2 * -cam_py} 0" rpy="0 0 0" />-->
 	  <origin xyz="0 0 0" rpy="0 0 0" />
 	  <parent link="camera_rgb_frame" />

File: costar_simulation/robot/kinect_properties2.xacro (robot description, xacro)
@@ -55,10 +55,3 @@
     </material>
   </xacro:property>
-	<property name="pi" value="3.14159265" />
-	<property name="cam_px" value="0" />
-<!--	<property name="cam_py" value="-0.0125" /> Y varies for different configurations. get sets in sensors_urdf -->
-	<property name="cam_pz" value="1" />
-	<property name="cam_or" value="0" />
-	<property name="cam_op" value="${pi*0.25}" />
-	<property name="cam_oy" value="0" />
 </robot>

Commit message: tweak kinect setup

File: costar_simulation/robot/kinect.xacro (robot description, xacro)
@@ -19,5 +19,5 @@
     <link name="camera_rgb_frame"/>
     <joint name="camera_rgb_optical_joint" type="fixed">
-      <origin xyz="0 0 0" rpy="${-M_PI/2} 0 ${-M_PI/2}" />
+      <origin xyz="0 ${-cam_py} 0" rpy="${-M_PI/2} 0 ${-M_PI/2}" />
       <parent link="camera_rgb_frame" />
       <child link="camera_rgb_optical_frame" />
@@ -25,5 +25,5 @@
     <link name="camera_rgb_optical_frame"/>
     <joint name="camera_joint" type="fixed">
-      <origin xyz="-0.031 ${-cam_py} -0.016" rpy="0 0 0"/>
+      <origin xyz="-0.031 0 -0.016" rpy="0 0 0"/>
       <parent link="camera_rgb_frame"/>
       <child link="camera_link"/>

Commit message: setting up start script

File: costar_simulation/robot/kinect.xacro (robot description, xacro)
@@ -4,5 +4,5 @@
   <xacro:include filename="$(find costar_simulation)/robot/kinect_properties2.xacro"/>
 	<property name="pi" value="3.14159265" />
-	<property name="cam_px" value="1.0" />
+	<property name="cam_px" value="0.0" />
   <property name="cam_py" value="1.0"/>
 	<property name="cam_pz" value="1.0" />
@@ -19,5 +19,5 @@
     <link name="camera_rgb_frame"/>
     <joint name="camera_rgb_optical_joint" type="fixed">
-      <origin xyz="0 ${-cam_py} 0" rpy="${-M_PI/2} 0 ${-M_PI/2}" />
+      <origin xyz="0 0 0" rpy="${-M_PI/2} 0 ${-M_PI/2}" />
       <parent link="camera_rgb_frame" />
       <child link="camera_rgb_optical_frame" />

Commit message: remove meshes

File: costar_simulation/robot/kinect.xacro (robot description, xacro)
@@ -33,5 +33,5 @@
        <origin xyz="0 0 0" rpy="0 0 ${M_PI/2}"/>
         <geometry>
-         <mesh filename="package://ur5_barrett_description/meshes/kinect/kinect.dae"/>
+         <mesh filename="package://costar_simulation/meshes/kinect/kinect.dae"/>
         </geometry>
       </visual>
