Commit message: add ur5 robot grasp link

File: costar_simulation/robot/ur5_joint_limited_robot.xacro (robot description, xacro)
@@ -14,3 +14,10 @@
     <origin xyz="0.0 0.0 0.0" rpy="${M_PI / 2} 0 0"/>
   </xacro:robotiq_85_gripper>
+  <!-- Create a grasp link to specify the end of the robot arm -->
+  <link name="grasp_link"/>
+  <joint name="ee_to_grasp_link" type="fixed">
+    <parent link="ee_link" />
+    <child link="grasp_link" />
+    <origin xyz="0.15 0.0 0.0" rpy="0 0 0"/>
+  </joint>
 </robot>
