Commit message: experimenting with robot setup for costar simulation

File: costar_simulation/robot/ur5_joint_limited_robot.urdf (robot description, URDF)
Before this commit: robot ur5_robotiq_parallel, 20 links, 19 joints
Links:
- removed link robotiq_85_base_link
- removed link robotiq_85_left_finger_link
- removed link robotiq_85_left_finger_tip_link
- removed link robotiq_85_left_inner_knuckle_link
- removed link robotiq_85_left_knuckle_link
- removed link robotiq_85_right_finger_link
- removed link robotiq_85_right_finger_tip_link
- removed link robotiq_85_right_inner_knuckle_link
- removed link robotiq_85_right_knuckle_link
- removed link robotiq_85_root
Joints:
- removed joint arm_to_gripper
- removed joint robotiq_85_base_joint
- removed joint robotiq_85_left_finger_joint
- removed joint robotiq_85_left_finger_tip_joint
- removed joint robotiq_85_left_inner_knuckle_joint
- removed joint robotiq_85_left_knuckle_joint
- removed joint robotiq_85_right_finger_joint
- removed joint robotiq_85_right_finger_tip_joint
- removed joint robotiq_85_right_inner_knuckle_joint
- removed joint robotiq_85_right_knuckle_joint

File: costar_simulation/robot/ur5_joint_limited_robot.xacro (robot description, xacro)
@@ -10,9 +10,9 @@
   <xacro:include filename="$(find ur5_robotiq_parallel_description)/urdf/robotiq_85/gripper.transmission.xacro" />
   <xacro:ur5_robot prefix="" joint_limited="true"/>
-  <xacro:robotiq_85_gripper prefix=""/>
+  <!--<xacro:robotiq_85_gripper prefix=""/>
   <joint name="arm_to_gripper" type="fixed">
     <parent link="ee_link"/>
     <child link="robotiq_85_root"/>
     <origin xyz="0 0 0" rpy="0 0 0"/>
-  </joint>
+  </joint>-->
 </robot>

Commit message: cleaning up definitions for ur5 robot

File: costar_simulation/robot/ur5_joint_limited_robot.urdf (robot description, URDF)
Before this commit: robot ur5_robotiq_parallel, 10 links, 9 joints
Links:
- link base_link: geometry collision mesh filename=package://costar_simulation/meshes/ur5/collision/base.stl; visual mesh filename=package://costar_simulation/meshes/ur5/visual/Base.dae.obj
- link forearm_link: geometry collision mesh filename=package://costar_simulation/meshes/ur5/collision/forearm.stl; visual mesh filename=package://costar_simulation/meshes/ur5/visual/Forearm.dae.o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
- link shoulder_link: geometry collision mesh filename=package://costar_simulation/meshes/ur5/collision/shoulder.s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; visual mesh filename=package://costar_simulation/meshes/ur5/visual/Shoulder.dae
- link upper_arm_link: geometry collision mesh filename=package://costar_simulation/meshes/ur5/collision/upper_arm.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; visual mesh filename=package://costar_simulation/meshes/ur5/visual/UpperArm.dae
- link wrist_1_link: geometry collision mesh filename=package://costar_simulation/meshes/ur5/collision/wrist_1.stl; visual mesh filename=package://costar_simulation/meshes/ur5/visual/Wrist1.dae
- link wrist_2_link: geometry collision mesh filename=package://costar_simulation/meshes/ur5/collision/wrist_2.stl; visual mesh filename=package://costar_simulation/meshes/ur5/visual/Wrist2.dae
- link wrist_3_link: geometry collision mesh filename=package://costar_simulation/meshes/ur5/collision/wrist_3.stl; visual mesh filename=package://costar_simulation/meshes/ur5/visual/Wrist3.dae

File: costar_simulation/robot/ur5_joint_limited_robot.xacro (robot description, xacro)
@@ -7,6 +7,6 @@
   <xacro:include filename="$(find costar_simulation)/robot/ur5/ur5.transmission.xacro" />
   <!-- Robotiq gripper -->
-  <xacro:include filename="$(find costar_simulation)/robot/robotiq_85/robotiq_85_gripper.urdf.xacro" />
-  <xacro:include filename="$(find costar_simulation)/robot/robotiq_85/gripper.transmission.xacro" />
+  <xacro:include filename="$(find costar_simulation)/robot/robotiq_85_gripper/urdf/robotiq_85_gripper.urdf.xacro" />
+  <xacro:include filename="$(find costar_simulation)/robot/robotiq_85_gripper/urdf/robotiq_85_gripper.transmission.xacro" />
   <xacro:ur5_robot prefix="" joint_limited="true"/>
   <!--<xacro:robotiq_85_gripper prefix=""/>

Commit message: adding all these sorting tasks

File: costar_simulation/robot/ur5_joint_limited_robot.urdf (robot description, URDF)
Before this commit: robot ur5_robotiq_parallel, 19 links, 18 joints
Joints:
- joint robotiq_85_right_knuckle_joint: mimic joint=robotiq_85_left_knuckle_joint -> joint=robotiq_85_left_knuckle_joint multiplier=1

Commit message: add grasp frame to robot

File: costar_simulation/robot/ur5_joint_limited_robot.urdf (robot description, URDF)
Before this commit: robot ur5_robotiq_parallel, 19 links, 18 joints
Links:
- added link grasp_link
Joints:
- added joint ee_to_grasp_link: type fixed, parent ee_link, child grasp_link, origin xyz=0.15 0.0 0.0 rpy=0 0 0
