Commit message: fix jaco robot

File: costar_simulation/robot/jaco_robot.urdf (robot description, URDF)
Before this commit: robot jaco_robot, 1 links, 0 joints
Links:
- added link jaco_0_baseA, mass 0.5688; collision mesh filename=package://jaco_description/meshes/jaco2/0_baseA.STL; visual mesh filename=package://jaco_description/meshes/jaco2/0_baseA.STL scale=0.98 0.98 0.98
- added link jaco_0_baseB_limb, mass 0.5152; collision mesh filename=package://jaco_description/meshes/jaco2/0_baseB_limb.STL; visual mesh filename=package://jaco_description/meshes/jaco2/0_baseB_limb.STL
- added link jaco_1_shoulder_limb, mass 0.4782; collision mesh filename=package://jaco_description/meshes/jaco2/1_shoulder_limb.STL; visual mesh filename=package://jaco_description/meshes/jaco2/1_shoulder_limb.STL
- added link jaco_2_upperarm_limb, mass 1.37163; collision mesh filename=package://jaco_description/meshes/jaco2/2_upperarm_limb.STL; visual mesh filename=package://jaco_description/meshes/jaco2/2_upperarm_limb.STL
- added link jaco_3_forearm_limb, mass 0.67592919; collision mesh filename=package://jaco_description/meshes/jaco2/3_forearm_limb.STL; visual mesh filename=package://jaco_description/meshes/jaco2/3_forearm_limb.STL
- added link jaco_4_upperwrist_limb, mass 0.24550336286; collision mesh filename=package://jaco_description/meshes/jaco2/4_upperwrist_limb.S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; visual mesh filename=package://jaco_description/meshes/jaco2/4_upperwrist_limb.S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
- added link jaco_5_lowerwrist_limb, mass 0.2455; collision mesh filename=package://jaco_description/meshes/jaco2/5_lowerwrist_limb.S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; visual mesh filename=package://jaco_description/meshes/jaco2/5_lowerwrist_limb.S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
- added link jaco_6_hand_limb, mass 0.2; collision mesh filename=package://jaco_description/meshes/jaco2/6_hand_limb.STL scale=1.0 1.0 1.0; visual mesh filename=package://jaco_description/meshes/jaco2/6_hand_limb.STL scale=1.0 1.0 1.0
- added link jaco_7_finger_mount_index, mass 0.006465; collision mesh filename=package://jaco_description/meshes/jaco2/7_finger_mount_inde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; visual mesh filename=package://jaco_description/meshes/jaco2/7_finger_mount_inde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
- added link jaco_7_finger_mount_pinkie, mass 0.00646; collision mesh filename=package://jaco_description/meshes/jaco2/7_finger_mount_pink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; visual mesh filename=package://jaco_description/meshes/jaco2/7_finger_mount_pink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
- added link jaco_7_finger_mount_thumb, mass 0.006465; collision mesh filename=package://jaco_description/meshes/jaco2/7_finger_mount_thum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; visual mesh filename=package://jaco_description/meshes/jaco2/7_finger_mount_thum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
- added link jaco_8_finger_index, mass 0.01845; collision mesh filename=package://jaco_description/meshes/jaco2/8_finger_index.STL; visual mesh filename=package://jaco_description/meshes/jaco2/8_finger_index.STL
- added link jaco_8_finger_pinkie, mass 0.01845; collision mesh filename=package://jaco_description/meshes/jaco2/8_finger_pinkie.STL; visual mesh filename=package://jaco_description/meshes/jaco2/8_finger_pinkie.STL
- added link jaco_8_finger_thumb, mass 0.0184; collision mesh filename=package://jaco_description/meshes/jaco2/8_finger_thumb.STL; visual mesh filename=package://jaco_description/meshes/jaco2/8_finger_thumb.STL
- added link jaco_9_finger_index_tip, mass 0.0122; collision mesh filename=package://jaco_description/meshes/jaco2/9_finger_index_tip.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 scale=1 1 1; visual mesh filename=package://jaco_description/meshes/jaco2/9_finger_index_tip.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 scale=1 1 1
- added link jaco_9_finger_pinkie_tip, mass 0.0122; collision mesh filename=package://jaco_description/meshes/jaco2/9_finger_pinkie_tip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 scale=1 1 1; visual mesh filename=package://jaco_description/meshes/jaco2/9_finger_pinkie_tip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 scale=1 1 1
- added link jaco_9_finger_thumb_tip, mass 0.0122; collision mesh filename=package://jaco_description/meshes/jaco2/9_finger_thumb_tip.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 scale=1 1 1; visual mesh filename=package://jaco_description/meshes/jaco2/9_finger_thumb_tip.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 scale=1 1 1
- added link jaco_fingers_base_link, mass 0.001
- added link jaco_ring_1, mass 0.00872; collision mesh filename=package://jaco_description/meshes/jaco2/ring_1.STL; visual mesh filename=package://jaco_description/meshes/jaco2/ring_1.STL
- added link jaco_ring_2, mass 0.00872; collision mesh filename=package://jaco_description/meshes/jaco2/ring_2.STL; visual mesh filename=package://jaco_description/meshes/jaco2/ring_2.STL
- added link jaco_ring_3, mass 0.00872; collision mesh filename=package://jaco_description/meshes/jaco2/ring_3.STL; visual mesh filename=package://jaco_description/meshes/jaco2/ring_3.STL
- added link jaco_ring_4, mass 0.00676534123969; collision mesh filename=package://jaco_description/meshes/jaco2/ring_4.STL; visual mesh filename=package://jaco_description/meshes/jaco2/ring_4.STL
- added link jaco_ring_5, mass 0.00676534123969; collision mesh filename=package://jaco_description/meshes/jaco2/ring_5.STL; visual mesh filename=package://jaco_description/meshes/jaco2/ring_5.STL
- added link jaco_ring_6, mass 0.00676; collision mesh filename=package://jaco_description/meshes/jaco2/ring_6.STL; visual mesh filename=package://jaco_description/meshes/jaco2/ring_6.STL
Joints:
- added joint jaco_arm_0_joint: type continuous, parent jaco_0_baseB_limb, child jaco_1_shoulder_limb, origin xyz=0 0.104 0 rpy=0 1.57079632679 0, axis 0 1 0, limit effort=8 velocity=1.0
- added joint jaco_arm_1_joint: type revolute, parent jaco_1_shoulder_limb, child jaco_2_upperarm_limb, origin xyz=0 0.1225 0 rpy=3.14159265359 -1.57079632679 0, axis 0 0 1, limit lower=-3.943 upper=0.81 effort=8 velocity=1.0
- added joint jaco_arm_2_joint: type revolute, parent jaco_2_upperarm_limb, child jaco_3_forearm_limb, origin xyz=0.41 0 0 rpy=0 0 1.57079632679489, axis 0 0 1, limit lower=-4.395 upper=1.252 effort=4 velocity=1.0
- added joint jaco_arm_3_joint: type continuous, parent jaco_3_forearm_limb, child jaco_4_upperwrist_limb, origin xyz=0.2073 0 0.0098 rpy=-1.57079632679484 0 -3.14159265358951, axis -1 0 0, limit effort=1.5 velocity=1.0
- added joint jaco_arm_4_joint: type continuous, parent jaco_4_upperwrist_limb, child jaco_5_lowerwrist_limb, origin xyz=-0.06590490 -0.034307921 0 rpy=0 0 0.959931089, axis -1 0 0, limit effort=1.0 velocity=1.0
- added joint jaco_arm_5_joint: type continuous, parent jaco_5_lowerwrist_limb, child jaco_6_hand_limb, origin xyz=-0.06590490 -0.034307921 0 rpy=-1.57079632679 0 0.959931089, axis -1 0 0, limit effort=1.0 velocity=1.0
- added joint jaco_arm_joint: type fixed, parent robot_root, child jaco_0_baseA, origin xyz=0 0 0 rpy=0 0 0
- added joint jaco_base_internal: type fixed, parent jaco_0_baseA, child jaco_0_baseB_limb, origin xyz=0 0 0.049 rpy=1.57079632679 0 0, axis 0 0 0
- added joint jaco_finger_joint_0: type revolute, parent jaco_fingers_base_link, child jaco_8_finger_index, origin xyz=-0.0276  0.0204 0.11 rpy=0 -0.34 -0.191986, axis 0 1 0, limit lower=-0.0045 upper=1.05 effort=1.5 velocity=0.2
- added joint jaco_finger_joint_1: type fixed, parent jaco_8_finger_index, child jaco_9_finger_index_tip, origin xyz=0 0 0.0441 rpy=0 0 0
- added joint jaco_finger_joint_2: type revolute, parent jaco_fingers_base_link, child jaco_8_finger_thumb, origin xyz= 0.0319  0.003  0.11 rpy=0 -0.37 2.91470065359, axis 0 1 0, limit lower=-0.0045 upper=1.05 effort=1.5 velocity=0.2
- added joint jaco_finger_joint_3: type fixed, parent jaco_8_finger_thumb, child jaco_9_finger_thumb_tip, origin xyz=0 0 0.0441 rpy=0 0 0
- added joint jaco_finger_joint_4: type revolute, parent jaco_fingers_base_link, child jaco_8_finger_pinkie, origin xyz=-0.0276 -0.0204 0.11 rpy=0 -0.34 0.191986, axis 0 1 0, limit lower=-0.0045 upper=1.05 effort=1.5 velocity=0.2
- added joint jaco_finger_joint_5: type fixed, parent jaco_8_finger_pinkie, child jaco_9_finger_pinkie_tip, origin xyz=0 0 0.0441 rpy=0 0 0
- added joint jaco_finger_mount_index_fixed: type fixed, parent jaco_fingers_base_link, child jaco_7_finger_mount_index, origin xyz=-0.034  0.022 0.095 rpy=0 -0.2293 -0.191986, axis 0 0 0
- added joint jaco_finger_mount_pinkie_fixed: type fixed, parent jaco_fingers_base_link, child jaco_7_finger_mount_pinkie, origin xyz=-0.034 -0.022 0.095 rpy=0 -0.2293 0.191986
- added joint jaco_finger_mount_thumb_fixed: type fixed, parent jaco_fingers_base_link, child jaco_7_finger_mount_thumb, origin xyz= 0.037  0.001  0.095 rpy=0 -0.2658 2.91470065359
- added joint jaco_fingers_base_joint: type fixed, parent jaco_6_hand_limb, child jaco_fingers_base_link, origin xyz=0 0 0 rpy=-1.57079632679 3.14159265359 1.57079632679
- added joint jaco_ring_1_joint: type fixed, parent jaco_0_baseB_limb, child jaco_ring_1, origin xyz=0 0.104 0 rpy=-1.57079632679 0.211499083190217 -3.14159265359, axis 0 0 0
- added joint jaco_ring_2_joint: type fixed, parent jaco_1_shoulder_limb, child jaco_ring_2, origin xyz=0 0.1225 0 rpy=-1.57079632679488 -1.49007956532211 1.57079632679488, axis 0 0 0
- added joint jaco_ring_3_joint: type fixed, parent jaco_2_upperarm_limb, child jaco_ring_3, origin xyz=0.41 0 0 rpy=3.14159265359 0 -3.14159265359, axis 0 0 0
- added joint jaco_ring_4_joint: type fixed, parent jaco_3_forearm_limb, child jaco_ring_4, origin xyz=0.2073 0 0.0098 rpy=3.14159265359 -1.57079632679 0, axis -1 0 0
- added joint jaco_ring_5_joint: type fixed, parent jaco_4_upperwrist_limb, child jaco_ring_5, origin xyz=-0.06590490 -0.034307921 0 rpy=-1.57079632679506 0 -0.610865238196312, axis -1 0 0
- added joint jaco_ring_6_joint: type fixed, parent jaco_5_lowerwrist_limb, child jaco_ring_6, origin xyz=-0.06590490 -0.034307921 0 rpy=1.57079632679 0 2.53072741539211 , axis 0 0 0

Commit message: add KDL inverse kinematics because pybullet IK wasn't doing the trick

File: costar_simulation/robot/jaco_robot.urdf (robot description, URDF)
Before this commit: robot jaco_robot, 25 links, 24 joints
Links:
- added link grasp_link
Joints:
- added joint ee_to_grasp_link: type fixed, parent jaco6_hand_limb, child grasp_link, origin xyz=0.15 0.0 0.0 rpy=0 0 0
