Commit message: adding kinect files for modification

File: costar_simulation/robot/ur5_joint_limited.xacro (robot description, xacro)
@@ -10,66 +10,73 @@
   <xacro:include filename="$(find ur5_robotiq_parallel_description)/urdf/robotiq_85/gripper.transmission.xacro" />
   <!-- Kinect -->
-   <xacro:include filename="$(find ur5_robotiq_parallel_description)/urdf/kinect/kinect.xacro"/>
-   <xacro:include filename="$(find ur5_robotiq_parallel_description)/urdf/kinect/kinect_properties2.xacro"/>
-   <xacro:include filename="$(find ur5_robotiq_parallel_description)/urdf/kinect/kinect_gazebo2.urdf.xacro"/>
- <property name="M_PI" value="3.14159"/>
-	<!-- property list -->
-	<xacro:property name="robot_stand_height" value="0.75"/>
-	<xacro:property name="kinect_stand_length" value="1.5"/>
-	<xacro:property name="kinect_stand_distance" value="0.10"/>
-	<xacro:ur5_robot prefix="" joint_limited="true"/>
-	<xacro:robotiq_85_gripper prefix=""/>
-	<!-- color macros -->
-	<xacro:macro name="material_orange_transparent">
-		<material name="orange_transparent">
-			<color rgba="1 0.5 0 0.4"/>
-		</material>
-	</xacro:macro>
-	<xacro:macro name="material_blue_transparent">
-		<material name="blue_transparent">
-			<color rgba="0 0.8 1 0.4"/>
-		</material>
-	</xacro:macro>
-	<xacro:material_orange_transparent />
-	<xacro:material_blue_transparent />
-	<!-- end of color macros -->
-	<link name="world"/>
-	<link name="stand">
-		<visual>
-		<geometry>
-		<cylinder radius="0.0735" length="${robot_stand_height}"/>
-		</geometry>
-		<material name="orange_transparent"/>
-		</visual>
-		<collision>
-		<geometry>
-		<cylinder radius="0.0735" length="${robot_stand_height}"/>
-		</geometry>
-		<material name="blue_transparent"/>
-		</collision>
-	</link>
-	<!-- instantiating sensor definitions -->
-	<!--sensor_kinect  parent="stand"/-->
-	<!-- end of sensor definitions -->
-	<!-- fixing barrett hand to the ur5 -->
-        <xacro:sensor_kinect  parent="stand" >
-     <!--origin xyz="0 1.8 0" rpy="0 0 0"/-->
-  </xacro:sensor_kinect >
-	<joint name="arm_to_gripper" type="fixed">
-		<parent link="ee_link"/>
-		<child link="robotiq_85_root"/>
-		<origin xyz="0 0 0" rpy="0 0 0"/>
-	</joint>
-	<!-- Hand attached to the arm -->
-	<joint name="world_to_stand" type="fixed">
-		<parent link="world"/>
-		<child link="stand"/>
-		<origin xyz="0 0 0" rpy="0 0 0"/>
-	</joint>
-	<joint name="stand_to_base" type="fixed">
-		<parent link="stand"/>
-		<!--child link="${arm_prefix}base_link"/-->
-		<child link="base_link"/>
-		<origin xyz="0 0 ${robot_stand_height * 0.5}" rpy="0 0 1.57"/>
-	</joint>
+  <xacro:include filename="$(find ur5_robotiq_parallel_description)/urdf/kinect/kinect.xacro"/>
+  <xacro:include filename="$(find ur5_robotiq_parallel_description)/urdf/kinect/kinect_properties2.xacro"/>
+  <xacro:include filename="$(find ur5_robotiq_parallel_description)/urdf/kinect/kinect_gazebo2.urdf.xacro"/>
+  <property name="M_PI" value="3.14159"/>
+  <!-- property list -->
+  <xacro:property name="robot_table_height" value="0.75"/>
+  <xacro:property name="robot_table_length" value="1.5"/>
+  <xacro:property name="robot_table_width" value="0.75"/>
+  <xacro:property name="kinect_table_length" value="1.5"/>
+  <xacro:property name="kinect_table_distance" value="0.10"/>
+  <xacro:property name="robot_name" value="ur5"/>
+  <xacro:ur5_robot prefix="" joint_limited="true"/>
+  <xacro:robotiq_85_gripper prefix=""/>
+  <!-- color macros -->
+  <xacro:macro name="material_orange_transparent">
+    <material name="orange_transparent">
+      <color rgba="1 0.5 0 0.4"/>
+    </material>
+  </xacro:macro>
+  <xacro:macro name="material_blue_transparent">
+    <material name="blue_transparent">
+      <color rgba="0 0.8 1 0.4"/>
+    </material>
+  </xacro:macro>
+  <xacro:material_orange_transparent />
+  <xacro:material_blue_transparent />
+  <!-- end of color macros -->
+  <link name="world"/>
+  <link name="table">
+    <visual>
+      <geometry>
+        <box size = "${robot_table_width} ${robot_table_length} ${robot_table_height}"/>
+        <cylinder radius="0.0735" length="${robot_table_height}"/>
+      </geometry>
+      <material name="orange_transparent"/>
+    </visual>
+    <collision>
+      <geometry>
+        <box size = "${robot_table_width} ${robot_table_length} ${robot_table_height}"/>
+      </geometry>
+      <material name="blue_transparent"/>
+    </collision>
+  </link>
+  <xacro:sensor_kinect  parent="table"/>
+  <joint name="arm_to_gripper" type="fixed">
+    <parent link="ee_link"/>
+    <child link="robotiq_85_root"/>
+    <origin xyz="0 0 0" rpy="0 0 0"/>
+  </joint>
+  <!-- Hand attached to the arm -->
+  <joint name="world_to_table" type="fixed">
+    <parent link="world"/>
+    <child link="table"/>
+    <origin xyz="0 0.75 0" rpy="0 0 0"/>
+  </joint>
+  <joint name="table_to_base" type="fixed">
+    <parent link="table"/>
+    <!--child link="${arm_prefix}base_link"/-->
+    <child link="base_link"/>
+    <origin xyz="0 0 ${robot_table_height * 0.5}" rpy="0 0 1.57"/>
+  </joint>
+  <!-- Create the planning scene for this world and publish it -->
+  <gazebo>
+    <plugin filename="libgazebo_ros_moveit_planning_scene.so" name="gazebo_ros_moveit_planning_scene">
+      <topicName>/planning_scene</topicName>
+      <sceneName>${robot_name}_scene</sceneName>
+      <robotName>${robot_name}</robotName>
+      <updatePeriod>0.01</updatePeriod>
+    </plugin>
+  </gazebo>
 </robot>

Commit message: setting up startup script

File: costar_simulation/robot/ur5_joint_limited.xacro (robot description, xacro)
@@ -15,4 +15,7 @@
   <property name="M_PI" value="3.14159"/>
   <!-- property list -->
+  <xacro:property name="robot_table_y" value="1.5"/>
+  <xacro:property name="robot_on_table_x" value="0.0"/>
+  <xacro:property name="robot_on_table_y" value="-0.5"/>
   <xacro:property name="robot_table_height" value="0.75"/>
   <xacro:property name="robot_table_length" value="1.5"/>
@@ -63,5 +66,5 @@
     <parent link="world"/>
     <child link="table"/>
-    <origin xyz="0 0.75 0" rpy="0 0 0"/>
+    <origin xyz="0 ${robot_table_y} 0" rpy="0 0 0"/>
   </joint>
   <joint name="table_to_base" type="fixed">
@@ -69,5 +72,5 @@
     <!--child link="${arm_prefix}base_link"/-->
     <child link="base_link"/>
-    <origin xyz="0 0 ${robot_table_height * 0.5}" rpy="0 0 1.57"/>
+    <origin xyz="${robot_on_table_x} ${robot_on_table_y} ${robot_table_height * 0.5}" rpy="0 0 1.57"/>
   </joint>
   <!-- Create the planning scene for this world and publish it -->

Commit message: fix startup

File: costar_simulation/robot/ur5_joint_limited.xacro (robot description, xacro)
@@ -72,5 +72,5 @@
     <!--child link="${arm_prefix}base_link"/-->
     <child link="base_link"/>
-    <origin xyz="${robot_on_table_x} ${robot_on_table_y} ${robot_table_height * 0.5}" rpy="0 0 1.57"/>
+    <origin xyz="${robot_on_table_x} ${robot_on_table_y} ${robot_table_height * 0.5}" rpy="0 0 -1.57"/>
   </joint>
   <!-- Create the planning scene for this world and publish it -->

Commit message: adding robotiq models

File: costar_simulation/robot/ur5_joint_limited.xacro (robot description, xacro)
@@ -7,6 +7,6 @@
   <xacro:include filename="$(find ur5_robotiq_parallel_description)/urdf/ur5/ur5.transmission.xacro" />
   <!-- Robotiq gripper -->
-  <xacro:include filename="$(find ur5_robotiq_parallel_description)/urdf/robotiq_85/robotiq_85_gripper.urdf.xacro" />
-  <xacro:include filename="$(find ur5_robotiq_parallel_description)/urdf/robotiq_85/gripper.transmission.xacro" />
+  <xacro:include filename="$(find costar_simulation)/robot/robotiq_85_gripper/urdf/robotiq_85_gripper.urdf.xacro" />
+  <xacro:include filename="$(find costar_simulation)/robot/robotiq_85_gripper/urdf/robotiq_85_gripper.transmission.xacro" />
   <!-- Kinect -->
   <xacro:include filename="$(find costar_simulation)/robot/kinect.xacro"/>
@@ -25,5 +25,7 @@
   <xacro:property name="robot_name" value="ur5"/>
   <xacro:ur5_robot prefix="" joint_limited="true"/>
-  <xacro:robotiq_85_gripper prefix=""/>
+  <xacro:robotiq_85_gripper prefix="" parent="ee_link">
+    <origin xyz="0.0 0.0 0.0" rpy="${M_PI / 2} 0 0"/>
+  </xacro:robotiq_85_gripper>
   <!-- color macros -->
   <xacro:macro name="material_orange_transparent">
@@ -57,9 +59,4 @@
   </link>
   <xacro:sensor_kinect  parent="table"/>
-  <joint name="arm_to_gripper" type="fixed">
-    <parent link="ee_link"/>
-    <child link="robotiq_85_root"/>
-    <origin xyz="0 0 0" rpy="0 0 0"/>
-  </joint>
   <!-- Hand attached to the arm -->
   <joint name="world_to_table" type="fixed">

Commit message: add a table

File: costar_simulation/robot/ur5_joint_limited.xacro (robot description, xacro)
@@ -1,4 +1,4 @@
 <?xml version="1.0" ?>
-<robot name="ur5_robotiq_parallel" xmlns:xacro="http://ros.org/wiki/xacro">
+<robot name="ur5" xmlns:xacro="http://ros.org/wiki/xacro">
   <!-- common stuff -->
   <xacro:include filename="$(find costar_simulation)/robot/ur5/ur5.gazebo.urdf.xacro" />
@@ -13,4 +13,6 @@
   <xacro:include filename="$(find costar_simulation)/robot/kinect_properties2.xacro"/>
   <xacro:include filename="$(find costar_simulation)/robot/kinect_gazebo2.urdf.xacro"/>
+  <!-- Table -->
+  <xacro:include filename="$(find costar_simulation)/urdf/table/table.xacro"/>
   <property name="M_PI" value="3.14159"/>
   <!-- property list -->
@@ -43,5 +45,5 @@
   <!-- end of color macros -->
   <link name="world"/>
-  <link name="table">
+  <!--<link name="table">
     <visual>
       <geometry>
@@ -57,5 +59,6 @@
       <material name="blue_transparent"/>
     </collision>
-  </link>
+  </link>-->
+  <xacro:table name="table"/>
   <xacro:sensor_kinect  parent="table"/>
   <!-- Hand attached to the arm -->

Commit message: revising bugs

File: costar_simulation/robot/ur5_joint_limited.xacro (robot description, xacro)
@@ -45,5 +45,5 @@
   <!-- end of color macros -->
   <link name="world"/>
-  <!--<link name="table">
+  <link name="table">
     <visual>
       <geometry>
@@ -59,6 +59,5 @@
       <material name="blue_transparent"/>
     </collision>
-  </link>-->
-  <xacro:table name="table"/>
+  </link>
   <xacro:sensor_kinect  parent="table"/>
   <!-- Hand attached to the arm -->

Commit message: update gazebo sim

File: costar_simulation/robot/ur5_joint_limited.xacro (robot description, xacro)
@@ -49,5 +49,5 @@
       <geometry>
         <box size = "${robot_table_width} ${robot_table_length} ${robot_table_height}"/>
-        <cylinder radius="0.0735" length="${robot_table_height}"/>
+        <!--<cylinder radius="0.0735" length="${robot_table_height}"/>-->
       </geometry>
       <material name="orange_transparent"/>
@@ -65,5 +65,5 @@
     <parent link="world"/>
     <child link="table"/>
-    <origin xyz="0 ${robot_table_y} 0" rpy="0 0 0"/>
+    <origin xyz="0 ${robot_table_y} ${robot_table_height * 0.5}" rpy="0 0 0"/>
   </joint>
   <joint name="table_to_base" type="fixed">
