Commit message: fix prereqs and force simulation to start in ROS mode for now

File: costar_simulation/robot/ur5/ur5.urdf.xacro (robot description, xacro)
@@ -72,5 +72,5 @@
       <visual>
         <geometry>
-          <mesh filename="package://costar_simulation/meshes/ur5/visual/Base.dae" />
+          <mesh filename="package://costar_simulation/meshes/ur5/visual/Base.dae.obj" />
         </geometry>
         <material name="LightGrey">
@@ -165,5 +165,5 @@
       <visual>
         <geometry>
-          <mesh filename="package://costar_simulation/meshes/ur5/visual/Forearm.dae" />
+          <mesh filename="package://costar_simulation/meshes/ur5/visual/Forearm.dae.obj" />
         </geometry>
         <material name="LightGrey">

Commit message: fixing issues with mesh position and alignment

File: costar_simulation/robot/ur5/ur5.urdf.xacro (robot description, xacro)
@@ -71,4 +71,5 @@
     <link name="${prefix}base_link" >
       <visual>
+        <origin rpy="${0.5 * pi} 0 0" xyz="0.0 0.0 0.0"/>
         <geometry>
           <mesh filename="package://costar_simulation/meshes/ur5/visual/Base.dae.obj" />
@@ -164,4 +165,5 @@
     <link name="${prefix}forearm_link">
       <visual>
+        <origin rpy="${0.5 * pi} 0 0" xyz="0.0 0.0 0.0"/>
         <geometry>
           <mesh filename="package://costar_simulation/meshes/ur5/visual/Forearm.dae.obj" />

Commit message: update xacro to define ur5 with robotiq 85 gripper

File: costar_simulation/robot/ur5/ur5.urdf.xacro (robot description, xacro)
@@ -103,6 +103,7 @@
     <link name="${prefix}shoulder_link">
       <visual>
-        <geometry>
-          <mesh filename="package://costar_simulation/meshes/ur5/visual/Shoulder.dae" />
+        <origin rpy="${0.5 * pi} 0 0" xyz="0.0 0.0 0.0"/>
+        <geometry>
+          <mesh filename="package://costar_simulation/meshes/ur5/visual/Shoulder.dae.obj" />
         </geometry>
         <material name="LightGrey">
@@ -134,6 +135,7 @@
     <link name="${prefix}upper_arm_link">
       <visual>
-        <geometry>
-          <mesh filename="package://costar_simulation/meshes/ur5/visual/UpperArm.dae" />
+        <origin rpy="${0.5 * pi} 0 0" xyz="0.0 0.0 0.0"/>
+        <geometry>
+          <mesh filename="package://costar_simulation/meshes/ur5/visual/UpperArm.dae.obj" />
         </geometry>
         <material name="LightGrey">
@@ -197,6 +199,7 @@
     <link name="${prefix}wrist_1_link">
       <visual>
-        <geometry>
-          <mesh filename="package://costar_simulation/meshes/ur5/visual/Wrist1.dae" />
+        <origin rpy="${0.5 * pi} 0 0" xyz="0.0 0.0 0.0"/>
+        <geometry>
+          <mesh filename="package://costar_simulation/meshes/ur5/visual/Wrist1.dae.obj" />
         </geometry>
         <material name="LightGrey">
@@ -228,6 +231,7 @@
     <link name="${prefix}wrist_2_link">
       <visual>
-        <geometry>
-          <mesh filename="package://costar_simulation/meshes/ur5/visual/Wrist2.dae" />
+        <origin rpy="${0.5 * pi} 0 0" xyz="0.0 0.0 0.0"/>
+        <geometry>
+          <mesh filename="package://costar_simulation/meshes/ur5/visual/Wrist2.dae.obj" />
         </geometry>
         <material name="LightGrey">
@@ -259,6 +263,7 @@
     <link name="${prefix}wrist_3_link">
       <visual>
-        <geometry>
-          <mesh filename="package://costar_simulation/meshes/ur5/visual/Wrist3.dae" />
+        <origin rpy="${0.5 * pi} 0 0" xyz="0.0 0.0 0.0"/>
+        <geometry>
+          <mesh filename="package://costar_simulation/meshes/ur5/visual/Wrist3.dae.obj" />
         </geometry>
         <material name="LightGrey">

File: costar_simulation/robot/ur5_joint_limited_robot.urdf (robot description, URDF)
Before this commit: robot ur5_robotiq_parallel, 10 links, 9 joints
Links:
- added link robotiq_85_base_link, mass 0.636951; collision mesh filename=package://costar_simulation/robot/robotiq_85_gripper/meshes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; visual mesh filename=package://costar_simulation/robot/robotiq_85_gripper/meshes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
- added link robotiq_85_left_finger_link, mass 0.027309; collision mesh filename=package://costar_simulation/robot/robotiq_85_gripper/meshes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; visual mesh filename=package://costar_simulation/robot/robotiq_85_gripper/meshes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
- added link robotiq_85_left_finger_tip_link, mass 0.019555; collision mesh filename=package://costar_simulation/robot/robotiq_85_gripper/meshes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; visual mesh filename=package://costar_simulation/robot/robotiq_85_gripper/meshes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
- added link robotiq_85_left_inner_knuckle_link, mass 0.029951; collision mesh filename=package://costar_simulation/robot/robotiq_85_gripper/meshes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; visual mesh filename=package://costar_simulation/robot/robotiq_85_gripper/meshes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
- added link robotiq_85_left_knuckle_link, mass 0.018491; collision mesh filename=package://costar_simulation/robot/robotiq_85_gripper/meshes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; visual mesh filename=package://costar_simulation/robot/robotiq_85_gripper/meshes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
- added link robotiq_85_right_finger_link, mass 0.027309; collision mesh filename=package://costar_simulation/robot/robotiq_85_gripper/meshes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; visual mesh filename=package://costar_simulation/robot/robotiq_85_gripper/meshes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
- added link robotiq_85_right_finger_tip_link, mass 0.019555; collision mesh filename=package://costar_simulation/robot/robotiq_85_gripper/meshes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; visual mesh filename=package://costar_simulation/robot/robotiq_85_gripper/meshes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
- added link robotiq_85_right_inner_knuckle_link, mass 0.029951; collision mesh filename=package://costar_simulation/robot/robotiq_85_gripper/meshes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; visual mesh filename=package://costar_simulation/robot/robotiq_85_gripper/meshes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
- added link robotiq_85_right_knuckle_link, mass 0.018491; collision mesh filename=package://costar_simulation/robot/robotiq_85_gripper/meshes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; visual mesh filename=package://costar_simulation/robot/robotiq_85_gripper/meshes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
- link shoulder_link: geometry collision mesh filename=package://costar_simulation/meshes/ur5/collision/shoulder.s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; visual mesh filename=package://costar_simulation/meshes/ur5/visual/Shoulder.dae.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
- link upper_arm_link: geometry collision mesh filename=package://costar_simulation/meshes/ur5/collision/upper_arm.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; visual mesh filename=package://costar_simulation/meshes/ur5/visual/UpperArm.dae.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
- link wrist_1_link: geometry collision mesh filename=package://costar_simulation/meshes/ur5/collision/wrist_1.stl; visual mesh filename=package://costar_simulation/meshes/ur5/visual/Wrist1.dae.obj
- link wrist_2_link: geometry collision mesh filename=package://costar_simulation/meshes/ur5/collision/wrist_2.stl; visual mesh filename=package://costar_simulation/meshes/ur5/visual/Wrist2.dae.obj
- link wrist_3_link: geometry collision mesh filename=package://costar_simulation/meshes/ur5/collision/wrist_3.stl; visual mesh filename=package://costar_simulation/meshes/ur5/visual/Wrist3.dae.obj
Joints:
- added joint robotiq_85_base_joint: type fixed, parent ee_link, child robotiq_85_base_link, origin xyz=0.0 0.0 0.0 rpy=1.570795 0 0
- added joint robotiq_85_left_finger_joint: type fixed, parent robotiq_85_left_knuckle_link, child robotiq_85_left_finger_link, origin xyz=-0.00408552455 -0.03148604435 0.0 rpy=0 0 0
- added joint robotiq_85_left_finger_tip_joint: type continuous, parent robotiq_85_left_inner_knuckle_link, child robotiq_85_left_finger_tip_link, origin xyz=0.04303959807 -0.03759940821 0.0 rpy=0.0 0.0 0.0, axis 0 0 1, limit lower=-3.14 upper=3.14 effort=0.1 velocity=100.0, mimic joint=robotiq_85_left_knuckle_joint multiplier=-1
- added joint robotiq_85_left_inner_knuckle_joint: type continuous, parent robotiq_85_base_link, child robotiq_85_left_inner_knuckle_link, origin xyz=0.06142 0.0127 0 rpy=3.14159 0.0 0.0, axis 0 0 1, limit lower=-3.14 upper=3.14 effort=0.1 velocity=100.0, mimic joint=robotiq_85_left_knuckle_joint offset=0
- added joint robotiq_85_left_knuckle_joint: type revolute, parent robotiq_85_base_link, child robotiq_85_left_knuckle_link, origin xyz=0.05490451627 0.03060114443 0.0 rpy=3.14159 0.0 0.0, axis 0 0 1, limit lower=0.0 upper=0.804 effort=1000 velocity=2.0
- added joint robotiq_85_right_finger_joint: type fixed, parent robotiq_85_right_knuckle_link, child robotiq_85_right_finger_link, origin xyz=-0.00408552455 -0.03148604435 0.0 rpy=0 0 0
- added joint robotiq_85_right_finger_tip_joint: type continuous, parent robotiq_85_right_inner_knuckle_link, child robotiq_85_right_finger_tip_link, origin xyz=0.04303959807 -0.03759940821  0.0 rpy=0.0 0.0 0.0, axis 0 0 1, limit lower=-3.14 upper=3.14 effort=0.1 velocity=100.0, mimic joint=robotiq_85_left_knuckle_joint multiplier=-1
- added joint robotiq_85_right_inner_knuckle_joint: type continuous, parent robotiq_85_base_link, child robotiq_85_right_inner_knuckle_link, origin xyz=0.06142 -0.0127 0 rpy=0 0 0, axis 0 0 1, limit lower=-3.14 upper=3.14 effort=0.1 velocity=100.0, mimic joint=robotiq_85_left_knuckle_joint offset=0
- added joint robotiq_85_right_knuckle_joint: type continuous, parent robotiq_85_base_link, child robotiq_85_right_knuckle_link, origin xyz=0.05490451627 -0.03060114443 0.0 rpy=0.0 0.0 0.0, axis 0 0 1, limit lower=-3.14 upper=3.14 effort=1000 velocity=100.0, mimic joint=robotiq_85_left_knuckle_joint

File: costar_simulation/robot/ur5_joint_limited_robot.xacro (robot description, xacro)
@@ -1,4 +1,5 @@
 <?xml version="1.0" ?>
 <robot name="ur5_robotiq_parallel" xmlns:xacro="http://ros.org/wiki/xacro">
+  <property name="M_PI" value="3.14159"/>
   <!-- common stuff -->
   <xacro:include filename="$(find costar_simulation)/robot/ur5/ur5.gazebo.urdf.xacro" />
@@ -10,9 +11,6 @@
   <xacro:include filename="$(find costar_simulation)/robot/robotiq_85_gripper/urdf/robotiq_85_gripper.transmission.xacro" />
   <xacro:ur5_robot prefix="" joint_limited="true"/>
-  <!--<xacro:robotiq_85_gripper prefix=""/>
-  <joint name="arm_to_gripper" type="fixed">
-    <parent link="ee_link"/>
-    <child link="robotiq_85_root"/>
-    <origin xyz="0 0 0" rpy="0 0 0"/>
-  </joint>-->
+  <xacro:robotiq_85_gripper prefix="" parent="ee_link">
+    <origin xyz="0.0 0.0 0.0" rpy="${M_PI / 2} 0 0"/>
+  </xacro:robotiq_85_gripper>
 </robot>

Commit message: fix issues with ur5 and bullet3 sim

File: costar_simulation/robot/ur5/ur5.urdf.xacro (robot description, xacro)
@@ -292,9 +292,17 @@
         <origin rpy="0 0 0" xyz="-0.01 0 0"/>
       </collision>
+      <xacro:cylinder_inertial radius="0.01" length="0.01" mass="0.0">
+        <origin xyz="0.0 0.0 0.0" rpy="0 0 0" />
+      </xacro:cylinder_inertial>
     </link>
     <xacro:ur5_arm_transmission prefix="${prefix}" />
     <xacro:ur5_arm_gazebo prefix="${prefix}" />
     <!-- ROS base_link to UR 'Base' Coordinates transform -->
-    <link name="${prefix}base"/>
+    <link name="${prefix}base">
+      <!-- add a tiny, zero-mass link -->
+      <xacro:cylinder_inertial radius="0.01" length="0.01" mass="0.0">
+        <origin xyz="0.0 0.0 0.0" rpy="0 0 0" />
+      </xacro:cylinder_inertial>
+    </link>
     <joint name="${prefix}base_link-base_fixed_joint" type="fixed">
       <!-- NOTE: this rotation is only needed as long as base_link itself is
@@ -307,5 +315,9 @@
     </joint>
     <!-- Frame coincident with all-zeros TCP on UR controller -->
-    <link name="${prefix}tool0"/>
+    <link name="${prefix}tool0">
+      <xacro:cylinder_inertial radius="0.01" length="0.01" mass="0.0">
+        <origin xyz="0.0 0.0 0.0" rpy="0 0 0" />
+      </xacro:cylinder_inertial>
+    </link>
     <joint name="${prefix}wrist_3_link-tool0_fixed_joint" type="fixed">
       <origin xyz="0 ${wrist_3_length} 0" rpy="${pi/-2.0} 0 0"/>

File: costar_simulation/robot/ur5_joint_limited_robot.xacro (robot description, xacro)
@@ -15,5 +15,9 @@
   </xacro:robotiq_85_gripper>
   <!-- Create a grasp link to specify the end of the robot arm -->
-  <link name="grasp_link"/>
+  <link name="grasp_link">
+    <xacro:cylinder_inertial radius="0.01" length="0.01" mass="0.0">
+      <origin xyz="0.0 0.0 0.0" rpy="0 0 0" />
+    </xacro:cylinder_inertial>
+  </link>
   <joint name="ee_to_grasp_link" type="fixed">
     <parent link="ee_link" />
