Commit message: tweaking robot setup

File: costar_simulation/robot/robotiq_85_gripper/urdf/robotiq_85_gripper.urdf.xacro (robot description, xacro)
@@ -41,5 +41,5 @@
             <origin rpy="0.0 0.0 0.0" xyz="0.05490451627 -0.03060114443 0.0"/>
             <limit lower="-3.14" upper="3.14" velocity="100.0" effort="1000"/>
-            <mimic joint="${prefix}robotiq_85_left_knuckle_joint"/>
+            <mimic joint="${prefix}robotiq_85_left_knuckle_joint" multiplier="1"/>
         </joint>
         <link name="${prefix}robotiq_85_left_knuckle_link">

Commit message: gripper commands and hacks to make them work better

File: costar_simulation/robot/robotiq_85_gripper/urdf/robotiq_85_gripper.urdf.xacro (robot description, xacro)
@@ -97,4 +97,5 @@
                 </geometry>
             </visual>
+            <!-- TODO(cpaxton): re-enable this
             <collision>
                 <geometry>
@@ -102,4 +103,5 @@
                 </geometry>
             </collision>
+            -->
             <inertial>
                 <mass value="0.027309" />
@@ -116,4 +118,5 @@
                 </geometry>
             </visual>
+            <!-- TODO(cpaxton): re-enable this
             <collision>
                 <geometry>
@@ -121,4 +124,5 @@
                 </geometry>
             </collision>
+            -->
             <inertial>
                 <mass value="0.027309" />

File: costar_simulation/robot/ur5_joint_limited_robot.urdf (robot description, URDF)
Before this commit: robot ur5_robotiq_parallel, 19 links, 18 joints
Links:
- link robotiq_85_left_finger_link: geometry visual mesh filename=package://costar_simulation/robot/robotiq_85_gripper/meshes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
- link robotiq_85_right_finger_link: geometry visual mesh filename=package://costar_simulation/robot/robotiq_85_gripper/meshes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

Commit message: add coliision mesh back in

File: costar_simulation/robot/robotiq_85_gripper/urdf/robotiq_85_gripper.urdf.xacro (robot description, xacro)
@@ -97,5 +97,4 @@
                 </geometry>
             </visual>
-            <!-- TODO(cpaxton): re-enable this
             <collision>
                 <geometry>
@@ -103,5 +102,4 @@
                 </geometry>
             </collision>
-            -->
             <inertial>
                 <mass value="0.027309" />
@@ -118,5 +116,4 @@
                 </geometry>
             </visual>
-            <!-- TODO(cpaxton): re-enable this
             <collision>
                 <geometry>
@@ -124,5 +121,4 @@
                 </geometry>
             </collision>
-            -->
             <inertial>
                 <mass value="0.027309" />

File: costar_simulation/robot/ur5_joint_limited_robot.urdf (robot description, URDF)
Before this commit: robot ur5_robotiq_parallel, 19 links, 18 joints
Links:
- link robotiq_85_left_finger_link: geometry collision mesh filename=package://costar_simulation/robot/robotiq_85_gripper/meshes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; visual mesh filename=package://costar_simulation/robot/robotiq_85_gripper/meshes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
- link robotiq_85_right_finger_link: geometry collision mesh filename=package://costar_simulation/robot/robotiq_85_gripper/meshes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; visual mesh filename=package://costar_simulation/robot/robotiq_85_gripper/meshes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
