Commit message: adding gripper geometry

File: costar_simulation/robot/robotiq_85_gripper/urdf/robotiq_85_gripper.urdf.xacro (robot description, xacro)
@@ -2,240 +2,249 @@
 <robot name="robotiq_85_gripper" xmlns:xacro="http://ros.org/wiki/xacro">
   <xacro:include filename="$(find costar_simulation)/robot/robotiq_85_gripper/urdf/robotiq_85_gripper.transmission.xacro" />
-    <property name="pi" value="3.14159"/>
-    <xacro:macro name="robotiq_85_gripper" params="prefix parent *origin">
-        <joint name="${prefix}robotiq_85_base_joint" type="fixed">
-            <parent link="${parent}"/>
-            <child link="${prefix}robotiq_85_base_link"/>
-            <xacro:insert_block name="origin"/>
-        </joint>
-        <link name="${prefix}robotiq_85_base_link">
-            <visual>
-                <geometry>
-                    <mesh filename="package://costar_simulation/robot/robotiq_85_gripper/meshes/visual/robotiq_85_base_link.dae"/>
-                </geometry>
-            </visual>
-            <collision>
-                <geometry>
-                    <mesh filename="package://costar_simulation/robot/robotiq_85_gripper/meshes/collision/robotiq_85_base_link.stl"/>
-                </geometry>
-            </collision>
-            <inertial>
-                <mass value="0.636951" />
-                <origin xyz="0.0 0.0 0.0" />
-                <inertia ixx = "0.000380" ixy = "0.000000" ixz = "0.000000"
-                         iyx = "0.000000" iyy = "0.001110" iyz = "0.000000"
-                         izx = "0.000000" izy = "0.000000" izz = "0.001171" />
-            </inertial>
-        </link>
-        <joint name="${prefix}robotiq_85_left_knuckle_joint" type="revolute">
-            <parent link="${prefix}robotiq_85_base_link"/>
-            <child link="${prefix}robotiq_85_left_knuckle_link"/>
-            <axis xyz="0 0 1"/>
-            <origin rpy="${pi} 0.0 0.0" xyz="0.05490451627 0.03060114443 0.0"/>
-            <limit lower="0.0" upper="0.804" velocity="2.0" effort="1000"/>
-        </joint>
-        <joint name="${prefix}robotiq_85_right_knuckle_joint" type="continuous">
-            <parent link="${prefix}robotiq_85_base_link"/>
-            <child link="${prefix}robotiq_85_right_knuckle_link"/>
-            <axis xyz="0 0 1"/>
-            <origin rpy="0.0 0.0 0.0" xyz="0.05490451627 -0.03060114443 0.0"/>
-            <limit lower="-3.14" upper="3.14" velocity="100.0" effort="1000"/>
-            <mimic joint="${prefix}robotiq_85_left_knuckle_joint" multiplier="1"/>
-        </joint>
-        <link name="${prefix}robotiq_85_left_knuckle_link">
-            <visual>
-                <geometry>
-                    <mesh filename="package://costar_simulation/robot/robotiq_85_gripper/meshes/visual/robotiq_85_knuckle_link.dae"/>
-                </geometry>
-            </visual>
-            <collision>
-                <geometry>
-                    <mesh filename="package://costar_simulation/robot/robotiq_85_gripper/meshes/collision/robotiq_85_knuckle_link.stl"/>
-                </geometry>
-            </collision>
-            <inertial>
-                <mass value="0.018491" />
-                <origin xyz="0.0 0.0 0.0" />
-                <inertia ixx = "0.000009" ixy = "-0.000001" ixz = "0.000000"
-                         iyx = "-0.000001" iyy = "0.000001" iyz = "0.000000"
-                         izx = "0.000000" izy = "0.000000" izz = "0.000010" />
-            </inertial>
-        </link>
-        <link name="${prefix}robotiq_85_right_knuckle_link">
-            <visual>
-                <geometry>
-                    <mesh filename="package://costar_simulation/robot/robotiq_85_gripper/meshes/visual/robotiq_85_knuckle_link.dae"/>
-                </geometry>
-            </visual>
-            <collision>
-                <geometry>
-                    <mesh filename="package://costar_simulation/robot/robotiq_85_gripper/meshes/collision/robotiq_85_knuckle_link.stl"/>
-                </geometry>
-            </collision>
-            <inertial>
-                <mass value="0.018491" />
-                <origin xyz="0.0 0.0 0.0" />
-                <inertia ixx = "0.000009" ixy = "-0.000001" ixz = "0.000000"
-                         iyx = "-0.000001" iyy = "0.000001" iyz = "0.000000"
-                         izx = "0.000000" izy = "0.000000" izz = "0.000010" />
-            </inertial>
-        </link>
-        <joint name="${prefix}robotiq_85_left_finger_joint" type="fixed">
-            <parent link="${prefix}robotiq_85_left_knuckle_link"/>
-            <child link="${prefix}robotiq_85_left_finger_link"/>
-            <origin xyz="-0.00408552455 -0.03148604435 0.0" rpy="0 0 0" />
-        </joint>
-        <joint name="${prefix}robotiq_85_right_finger_joint" type="fixed">
-            <parent link="${prefix}robotiq_85_right_knuckle_link"/>
-            <child link="${prefix}robotiq_85_right_finger_link"/>
-            <origin xyz="-0.00408552455 -0.03148604435 0.0" rpy="0 0 0" />
-        </joint>
-        <link name="${prefix}robotiq_85_left_finger_link">
-            <visual>
-                <geometry>
-                    <mesh filename="package://costar_simulation/robot/robotiq_85_gripper/meshes/visual/robotiq_85_finger_link.dae"/>
-                </geometry>
-            </visual>
-            <collision>
-                <geometry>
-                    <mesh filename="package://costar_simulation/robot/robotiq_85_gripper/meshes/collision/robotiq_85_finger_link.stl"/>
-                </geometry>
-            </collision>
-            <inertial>
-                <mass value="0.027309" />
-                <origin xyz="0.0 0.0 0.0" />
-                <inertia ixx = "0.000003" ixy = "-0.000002" ixz = "0.000000"
-                         iyx = "-0.000002" iyy = "0.000021" iyz = "0.000000"
-                         izx = "0.000000" izy = "0.000000" izz = "0.000020" />
-            </inertial>
-        </link>
-        <link name="${prefix}robotiq_85_right_finger_link">
-            <visual>
-                <geometry>
-                    <mesh filename="package://costar_simulation/robot/robotiq_85_gripper/meshes/visual/robotiq_85_finger_link.dae"/>
-                </geometry>
-            </visual>
-            <collision>
-                <geometry>
-                    <mesh filename="package://costar_simulation/robot/robotiq_85_gripper/meshes/collision/robotiq_85_finger_link.stl"/>
-                </geometry>
-            </collision>
-            <inertial>
-                <mass value="0.027309" />
-                <origin xyz="0.0 0.0 0.0" />
-                <inertia ixx = "0.000003" ixy = "-0.000002" ixz = "0.000000"
-                         iyx = "-0.000002" iyy = "0.000021" iyz = "0.000000"
-                         izx = "0.000000" izy = "0.000000" izz = "0.000020" />
-            </inertial>
-        </link>
-        <joint name="${prefix}robotiq_85_left_inner_knuckle_joint" type="continuous">
-            <parent link="${prefix}robotiq_85_base_link"/>
-            <child link="${prefix}robotiq_85_left_inner_knuckle_link"/>
-            <axis xyz="0 0 1"/>
-            <origin xyz="0.06142 0.0127 0" rpy="${pi} 0.0 0.0" />
-            <limit lower="-3.14" upper="3.14" velocity="100.0" effort="0.1"/>
-            <mimic joint="${prefix}robotiq_85_left_knuckle_joint" offset="0"/>
-        </joint>
-        <joint name="${prefix}robotiq_85_right_inner_knuckle_joint" type="continuous">
-            <parent link="${prefix}robotiq_85_base_link"/>
-            <child link="${prefix}robotiq_85_right_inner_knuckle_link"/>
-            <axis xyz="0 0 1"/>
-            <origin xyz="0.06142 -0.0127 0" rpy="0 0 0"/>
-            <limit lower="-3.14" upper="3.14" velocity="100.0" effort="0.1"/>
-            <mimic joint="${prefix}robotiq_85_left_knuckle_joint" offset="0"/>
-        </joint>
-        <link name="${prefix}robotiq_85_left_inner_knuckle_link">
-            <visual>
-                <geometry>
-                    <mesh filename="package://costar_simulation/robot/robotiq_85_gripper/meshes/visual/robotiq_85_inner_knuckle_link.dae"/>
-                </geometry>
-            </visual>
-            <collision>
-                <geometry>
-                    <mesh filename="package://costar_simulation/robot/robotiq_85_gripper/meshes/collision/robotiq_85_inner_knuckle_link.stl"/>
-                </geometry>
-            </collision>
-            <inertial>
-                <mass value="0.029951" />
-                <origin xyz="0.0 0.0 0.0" />
-                <inertia ixx = "0.000039" ixy = "0.000000" ixz = "0.000000"
-                         iyx = "0.000000" iyy = "0.000005" iyz = "0.000000"
-                         izx = "0.000000" izy = "0.000000" izz = "0.000035" />
-            </inertial>
-        </link>
-        <link name="${prefix}robotiq_85_right_inner_knuckle_link">
-            <visual>
-                <geometry>
-                    <mesh filename="package://costar_simulation/robot/robotiq_85_gripper/meshes/visual/robotiq_85_inner_knuckle_link.dae"/>
-                </geometry>
-            </visual>
-            <collision>
-                <geometry>
-                    <mesh filename="package://costar_simulation/robot/robotiq_85_gripper/meshes/collision/robotiq_85_inner_knuckle_link.stl"/>
-                </geometry>
-            </collision>
-            <inertial>
-                <mass value="0.029951" />
-                <origin xyz="0.0 0.0 0.0" />
-                <inertia ixx = "0.000039" ixy = "0.000000" ixz = "0.000000"
-                         iyx = "0.000000" iyy = "0.000005" iyz = "0.000000"
-                         izx = "0.000000" izy = "0.000000" izz = "0.000035" />
-            </inertial>
-        </link>
-        <joint name="${prefix}robotiq_85_left_finger_tip_joint" type="continuous">
-            <parent link="${prefix}robotiq_85_left_inner_knuckle_link"/>
-            <child link="${prefix}robotiq_85_left_finger_tip_link"/>
-            <axis xyz="0 0 1"/>
-            <origin xyz="0.04303959807 -0.03759940821 0.0" rpy="0.0 0.0 0.0"/>
-            <limit lower="-3.14" upper="3.14" velocity="100.0" effort="0.1"/>
-            <mimic joint="${prefix}robotiq_85_left_knuckle_joint" multiplier="-1"/>
-        </joint>
-        <joint name="${prefix}robotiq_85_right_finger_tip_joint" type="continuous">
-            <parent link="${prefix}robotiq_85_right_inner_knuckle_link"/>
-            <child link="${prefix}robotiq_85_right_finger_tip_link"/>
-            <axis xyz="0 0 1"/>
-            <origin rpy="0.0 0.0 0.0" xyz="0.04303959807 -0.03759940821  0.0"/>
-            <limit lower="-3.14" upper="3.14" velocity="100.0" effort="0.1"/>
-            <mimic joint="${prefix}robotiq_85_left_knuckle_joint" multiplier="-1"/>
-        </joint>
-        <link name="${prefix}robotiq_85_left_finger_tip_link">
-            <visual>
-                <geometry>
-                    <mesh filename="package://costar_simulation/robot/robotiq_85_gripper/meshes/visual/robotiq_85_finger_tip_link.dae"/>
-                </geometry>
-            </visual>
-            <collision>
-                <geometry>
-                    <mesh filename="package://costar_simulation/robot/robotiq_85_gripper/meshes/collision/robotiq_85_finger_tip_link.stl"/>
-                </geometry>
-            </collision>
-            <inertial>
-                <mass value="0.019555" />
-                <origin xyz="0.0 0.0 0.0" />
-                <inertia ixx = "0.000002" ixy = "0.000000" ixz = "0.000000"
-                         iyx = "0.000000" iyy = "0.000005" iyz = "0.000000"
-                         izx = "0.000000" izy = "0.000000" izz = "0.000006" />
-            </inertial>
-        </link>
-        <link name="${prefix}robotiq_85_right_finger_tip_link">
-            <visual>
-                <geometry>
-                    <mesh filename="package://costar_simulation/robot/robotiq_85_gripper/meshes/visual/robotiq_85_finger_tip_link.dae"/>
-                </geometry>
-            </visual>
-            <collision>
-                <geometry>
-                    <mesh filename="package://costar_simulation/robot/robotiq_85_gripper/meshes/collision/robotiq_85_finger_tip_link.stl"/>
-                </geometry>
-            </collision>
-            <inertial>
-                <mass value="0.019555" />
-                <origin xyz="0.0 0.0 0.0" />
-                <inertia ixx = "0.000002" ixy = "0.000000" ixz = "0.000000"
-                         iyx = "0.000000" iyy = "0.000005" iyz = "0.000000"
-                         izx = "0.000000" izy = "0.000000" izz = "0.000006" />
-            </inertial>
-        </link>
-        <xacro:robotiq_85_gripper_transmission prefix="${prefix}" />
-    </xacro:macro>
+  <property name="pi" value="3.14159"/>
+  <xacro:macro name="robotiq_85_gripper" params="prefix parent *origin">
+    <joint name="${prefix}robotiq_85_base_joint" type="fixed">
+      <parent link="${parent}"/>
+      <child link="${prefix}robotiq_85_base_link"/>
+      <xacro:insert_block name="origin"/>
+    </joint>
+    <link name="${prefix}robotiq_85_base_link">
+      <visual>
+        <origin rpy="${0.5 * pi} 0 0" xyz="0.0 0.0 0.0"/>
+        <geometry>
+          <mesh filename="package://costar_simulation/robot/robotiq_85_gripper/meshes/visual/robotiq_85_base_link.dae.obj"/>
+        </geometry>
+      </visual>
+      <collision>
+        <geometry>
+          <mesh filename="package://costar_simulation/robot/robotiq_85_gripper/meshes/collision/robotiq_85_base_link.stl"/>
+        </geometry>
+      </collision>
+      <inertial>
+        <mass value="0.636951" />
+        <origin xyz="0.0 0.0 0.0" />
+        <inertia ixx = "0.000380" ixy = "0.000000" ixz = "0.000000"
+          iyx = "0.000000" iyy = "0.001110" iyz = "0.000000"
+          izx = "0.000000" izy = "0.000000" izz = "0.001171" />
+      </inertial>
+    </link>
+    <joint name="${prefix}robotiq_85_left_knuckle_joint" type="revolute">
+      <parent link="${prefix}robotiq_85_base_link"/>
+      <child link="${prefix}robotiq_85_left_knuckle_link"/>
+      <axis xyz="0 0 1"/>
+      <origin rpy="${pi} 0.0 0.0" xyz="0.05490451627 0.03060114443 0.0"/>
+      <limit lower="0.0" upper="0.804" velocity="2.0" effort="1000"/>
+    </joint>
+    <joint name="${prefix}robotiq_85_right_knuckle_joint" type="continuous">
+      <parent link="${prefix}robotiq_85_base_link"/>
+      <child link="${prefix}robotiq_85_right_knuckle_link"/>
+      <axis xyz="0 0 1"/>
+      <origin rpy="0.0 0.0 0.0" xyz="0.05490451627 -0.03060114443 0.0"/>
+      <limit lower="-3.14" upper="3.14" velocity="100.0" effort="1000"/>
+      <mimic joint="${prefix}robotiq_85_left_knuckle_joint" multiplier="1"/>
+    </joint>
+    <link name="${prefix}robotiq_85_left_knuckle_link">
+      <visual>
+        <origin rpy="${0.5 * pi} 0 0" xyz="0.0 0.0 0.0"/>
+        <geometry>
+          <mesh filename="package://costar_simulation/robot/robotiq_85_gripper/meshes/visual/robotiq_85_knuckle_link.dae.obj"/>
+        </geometry>
+      </visual>
+      <collision>
+        <geometry>
+          <mesh filename="package://costar_simulation/robot/robotiq_85_gripper/meshes/collision/robotiq_85_knuckle_link.stl"/>
+        </geometry>
+      </collision>
+      <inertial>
+        <mass value="0.018491" />
+        <origin xyz="0.0 0.0 0.0" />
+        <inertia ixx = "0.000009" ixy = "-0.000001" ixz = "0.000000"
+          iyx = "-0.000001" iyy = "0.000001" iyz = "0.000000"
+          izx = "0.000000" izy = "0.000000" izz = "0.000010" />
+      </inertial>
+    </link>
+    <link name="${prefix}robotiq_85_right_knuckle_link">
+      <visual>
+        <origin rpy="${0.5 * pi} 0 0" xyz="0.0 0.0 0.0"/>
+        <geometry>
+          <mesh filename="package://costar_simulation/robot/robotiq_85_gripper/meshes/visual/robotiq_85_knuckle_link.dae.obj"/>
+        </geometry>
+      </visual>
+      <collision>
+        <geometry>
+          <mesh filename="package://costar_simulation/robot/robotiq_85_gripper/meshes/collision/robotiq_85_knuckle_link.stl"/>
+        </geometry>
+      </collision>
+      <inertial>
+        <mass value="0.018491" />
+        <origin xyz="0.0 0.0 0.0" />
+        <inertia ixx = "0.000009" ixy = "-0.000001" ixz = "0.000000"
+          iyx = "-0.000001" iyy = "0.000001" iyz = "0.000000"
+          izx = "0.000000" izy = "0.000000" izz = "0.000010" />
+      </inertial>
+    </link>
+    <joint name="${prefix}robotiq_85_left_finger_joint" type="fixed">
+      <parent link="${prefix}robotiq_85_left_knuckle_link"/>
+      <child link="${prefix}robotiq_85_left_finger_link"/>
+      <origin xyz="-0.00408552455 -0.03148604435 0.0" rpy="0 0 0" />
+    </joint>
+    <joint name="${prefix}robotiq_85_right_finger_joint" type="fixed">
+      <parent link="${prefix}robotiq_85_right_knuckle_link"/>
+      <child link="${prefix}robotiq_85_right_finger_link"/>
+      <origin xyz="-0.00408552455 -0.03148604435 0.0" rpy="0 0 0" />
+    </joint>
+    <link name="${prefix}robotiq_85_left_finger_link">
+      <visual>
+        <origin rpy="${0.5 * pi} 0 0" xyz="0.0 0.0 0.0"/>
+        <geometry>
+          <mesh filename="package://costar_simulation/robot/robotiq_85_gripper/meshes/visual/robotiq_85_finger_link.dae.obj"/>
+        </geometry>
+      </visual>
+      <collision>
+        <geometry>
+          <mesh filename="package://costar_simulation/robot/robotiq_85_gripper/meshes/collision/robotiq_85_finger_link.stl"/>
+        </geometry>
+      </collision>
+      <inertial>
+        <mass value="0.027309" />
+        <origin xyz="0.0 0.0 0.0" />
+        <inertia ixx = "0.000003" ixy = "-0.000002" ixz = "0.000000"
+          iyx = "-0.000002" iyy = "0.000021" iyz = "0.000000"
+          izx = "0.000000" izy = "0.000000" izz = "0.000020" />
+      </inertial>
+    </link>
+    <link name="${prefix}robotiq_85_right_finger_link">
+      <visual>
+        <origin rpy="${0.5 * pi} 0 0" xyz="0.0 0.0 0.0"/>
+        <geometry>
+          <mesh filename="package://costar_simulation/robot/robotiq_85_gripper/meshes/visual/robotiq_85_finger_link.dae.obj"/>
+        </geometry>
+      </visual>
+      <collision>
+        <geometry>
+          <mesh filename="package://costar_simulation/robot/robotiq_85_gripper/meshes/collision/robotiq_85_finger_link.stl"/>
+        </geometry>
+      </collision>
+      <inertial>
+        <mass value="0.027309" />
+        <origin xyz="0.0 0.0 0.0" />
+        <inertia ixx = "0.000003" ixy = "-0.000002" ixz = "0.000000"
+          iyx = "-0.000002" iyy = "0.000021" iyz = "0.000000"
+          izx = "0.000000" izy = "0.000000" izz = "0.000020" />
+      </inertial>
+    </link>
+    <joint name="${prefix}robotiq_85_left_inner_knuckle_joint" type="continuous">
+      <parent link="${prefix}robotiq_85_base_link"/>
+      <child link="${prefix}robotiq_85_left_inner_knuckle_link"/>
+      <axis xyz="0 0 1"/>
+      <origin xyz="0.06142 0.0127 0" rpy="${pi} 0.0 0.0" />
+      <limit lower="-3.14" upper="3.14" velocity="100.0" effort="0.1"/>
+      <mimic joint="${prefix}robotiq_85_left_knuckle_joint" offset="0"/>
+    </joint>
+    <joint name="${prefix}robotiq_85_right_inner_knuckle_joint" type="continuous">
+      <parent link="${prefix}robotiq_85_base_link"/>
+      <child link="${prefix}robotiq_85_right_inner_knuckle_link"/>
+      <axis xyz="0 0 1"/>
+      <origin xyz="0.06142 -0.0127 0" rpy="0 0 0"/>
+      <limit lower="-3.14" upper="3.14" velocity="100.0" effort="0.1"/>
+      <mimic joint="${prefix}robotiq_85_left_knuckle_joint" offset="0"/>
+    </joint>
+    <link name="${prefix}robotiq_85_left_inner_knuckle_link">
+      <visual>
+        <origin rpy="${0.5 * pi} 0 0" xyz="0.0 0.0 0.0"/>
+        <geometry>
+          <mesh filename="package://costar_simulation/robot/robotiq_85_gripper/meshes/visual/robotiq_85_inner_knuckle_link.dae.obj"/>
+        </geometry>
+      </visual>
+      <collision>
+        <geometry>
+          <mesh filename="package://costar_simulation/robot/robotiq_85_gripper/meshes/collision/robotiq_85_inner_knuckle_link.stl"/>
+        </geometry>
+      </collision>
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
Commit message: color for gripper

File: costar_simulation/robot/robotiq_85_gripper/urdf/robotiq_85_gripper.urdf.xacro (robot description, xacro)
@@ -3,4 +3,7 @@
   <xacro:include filename="$(find costar_simulation)/robot/robotiq_85_gripper/urdf/robotiq_85_gripper.transmission.xacro" />
   <property name="pi" value="3.14159"/>
+  <material name="blackish">
+    <color rgba="0.2 0.2 0.2 1"/>
+  </material>
   <xacro:macro name="robotiq_85_gripper" params="prefix parent *origin">
     <joint name="${prefix}robotiq_85_base_joint" type="fixed">
@@ -11,4 +14,5 @@
     <link name="${prefix}robotiq_85_base_link">
       <visual>
+        <material name="blackish"/>
         <origin rpy="${0.5 * pi} 0 0" xyz="0.0 0.0 0.0"/>
         <geometry>
@@ -46,4 +50,5 @@
     <link name="${prefix}robotiq_85_left_knuckle_link">
       <visual>
+        <material name="blackish"/>
         <origin rpy="${0.5 * pi} 0 0" xyz="0.0 0.0 0.0"/>
         <geometry>
@@ -66,4 +71,5 @@
     <link name="${prefix}robotiq_85_right_knuckle_link">
       <visual>
+        <material name="blackish"/>
         <origin rpy="${0.5 * pi} 0 0" xyz="0.0 0.0 0.0"/>
         <geometry>
@@ -96,4 +102,5 @@
     <link name="${prefix}robotiq_85_left_finger_link">
       <visual>
+        <material name="blackish"/>
         <origin rpy="${0.5 * pi} 0 0" xyz="0.0 0.0 0.0"/>
         <geometry>
@@ -116,4 +123,5 @@
     <link name="${prefix}robotiq_85_right_finger_link">
       <visual>
+        <material name="blackish"/>
         <origin rpy="${0.5 * pi} 0 0" xyz="0.0 0.0 0.0"/>
         <geometry>
@@ -152,4 +160,5 @@
     <link name="${prefix}robotiq_85_left_inner_knuckle_link">
       <visual>
+        <material name="blackish"/>
         <origin rpy="${0.5 * pi} 0 0" xyz="0.0 0.0 0.0"/>
         <geometry>
@@ -172,4 +181,5 @@
     <link name="${prefix}robotiq_85_right_inner_knuckle_link">
       <visual>
+        <material name="blackish"/>
         <origin rpy="${0.5 * pi} 0 0" xyz="0.0 0.0 0.0"/>
         <geometry>
@@ -208,4 +218,5 @@
     <link name="${prefix}robotiq_85_left_finger_tip_link">
       <visual>
+        <material name="blackish"/>
         <origin rpy="${0.5 * pi} 0 0" xyz="0.0 0.0 0.0"/>
         <geometry>
@@ -232,4 +243,5 @@
     <link name="${prefix}robotiq_85_right_finger_tip_link">
       <visual>
+        <material name="blackish"/>
         <origin rpy="${0.5 * pi} 0 0" xyz="0.0 0.0 0.0"/>
         <geometry>
