Commit message: modifying things so we can use gazebo instead of pybullet

File: costar_simulation/robot/robotiq_85_gripper/urdf/robotiq_85_gripper.urdf.xacro (robot description, xacro)
@@ -17,5 +17,5 @@
         <origin rpy="${0.5 * pi} 0 0" xyz="0.0 0.0 0.0"/>
         <geometry>
-          <mesh filename="package://costar_simulation/robot/robotiq_85_gripper/meshes/visual/robotiq_85_base_link.dae.obj"/>
+          <mesh filename="package://costar_simulation/robot/robotiq_85_gripper/meshes/visual/robotiq_85_base_link.dae"/>
         </geometry>
       </visual>
@@ -53,5 +53,5 @@
         <origin rpy="${0.5 * pi} 0 0" xyz="0.0 0.0 0.0"/>
         <geometry>
-          <mesh filename="package://costar_simulation/robot/robotiq_85_gripper/meshes/visual/robotiq_85_knuckle_link.dae.obj"/>
+          <mesh filename="package://costar_simulation/robot/robotiq_85_gripper/meshes/visual/robotiq_85_knuckle_link.dae"/>
         </geometry>
       </visual>
@@ -74,5 +74,5 @@
         <origin rpy="${0.5 * pi} 0 0" xyz="0.0 0.0 0.0"/>
         <geometry>
-          <mesh filename="package://costar_simulation/robot/robotiq_85_gripper/meshes/visual/robotiq_85_knuckle_link.dae.obj"/>
+          <mesh filename="package://costar_simulation/robot/robotiq_85_gripper/meshes/visual/robotiq_85_knuckle_link.dae"/>
         </geometry>
       </visual>
@@ -109,5 +109,5 @@
         <origin rpy="${0.5 * pi} 0 0" xyz="0.0 0.0 0.0"/>
         <geometry>
-          <mesh filename="package://costar_simulation/robot/robotiq_85_gripper/meshes/visual/robotiq_85_finger_link.dae.obj"/>
+          <mesh filename="package://costar_simulation/robot/robotiq_85_gripper/meshes/visual/robotiq_85_finger_link.dae"/>
         </geometry>
       </visual>
@@ -135,5 +135,5 @@
         <origin rpy="${0.5 * pi} 0 0" xyz="0.0 0.0 0.0"/>
         <geometry>
-          <mesh filename="package://costar_simulation/robot/robotiq_85_gripper/meshes/visual/robotiq_85_finger_link.dae.obj"/>
+          <mesh filename="package://costar_simulation/robot/robotiq_85_gripper/meshes/visual/robotiq_85_finger_link.dae"/>
         </geometry>
       </visual>
@@ -177,5 +177,5 @@
         <origin rpy="${0.5 * pi} 0 0" xyz="0.0 0.0 0.0"/>
         <geometry>
-          <mesh filename="package://costar_simulation/robot/robotiq_85_gripper/meshes/visual/robotiq_85_inner_knuckle_link.dae.obj"/>
+          <mesh filename="package://costar_simulation/robot/robotiq_85_gripper/meshes/visual/robotiq_85_inner_knuckle_link.dae"/>
         </geometry>
       </visual>
@@ -203,5 +203,5 @@
         <origin rpy="${0.5 * pi} 0 0" xyz="0.0 0.0 0.0"/>
         <geometry>
-          <mesh filename="package://costar_simulation/robot/robotiq_85_gripper/meshes/visual/robotiq_85_inner_knuckle_link.dae.obj"/>
+          <mesh filename="package://costar_simulation/robot/robotiq_85_gripper/meshes/visual/robotiq_85_inner_knuckle_link.dae"/>
         </geometry>
       </visual>
@@ -240,5 +240,5 @@
         <origin rpy="${0.5 * pi} 0 0" xyz="0.0 0.0 0.0"/>
         <geometry>
-          <mesh filename="package://costar_simulation/robot/robotiq_85_gripper/meshes/visual/robotiq_85_finger_tip_link.dae.obj"/>
+          <mesh filename="package://costar_simulation/robot/robotiq_85_gripper/meshes/visual/robotiq_85_finger_tip_link.dae"/>
         </geometry>
       </visual>
@@ -266,5 +266,5 @@
         <origin rpy="${0.5 * pi} 0 0" xyz="0.0 0.0 0.0"/>
         <geometry>
-          <mesh filename="package://costar_simulation/robot/robotiq_85_gripper/meshes/visual/robotiq_85_finger_tip_link.dae.obj"/>
+          <mesh filename="package://costar_simulation/robot/robotiq_85_gripper/meshes/visual/robotiq_85_finger_tip_link.dae"/>
         </geometry>
       </visual>

Commit message: Merge branch 'feature/sim-updates' of github.com:cpaxton/costar_plan into feature/sim-updates

File: costar_simulation/robot/robotiq_85_gripper/urdf/robotiq_85_gripper.urdf.xacro (robot description, xacro)
@@ -17,5 +17,5 @@
         <origin rpy="${0.5 * pi} 0 0" xyz="0.0 0.0 0.0"/>
         <geometry>
-          <mesh filename="package://costar_simulation/robot/robotiq_85_gripper/meshes/visual/robotiq_85_base_link.dae"/>
+          <mesh filename="package://costar_simulation/robot/robotiq_85_gripper/meshes/visual/robotiq_85_base_link.dae.obj"/>
         </geometry>
       </visual>
@@ -53,5 +53,5 @@
         <origin rpy="${0.5 * pi} 0 0" xyz="0.0 0.0 0.0"/>
         <geometry>
-          <mesh filename="package://costar_simulation/robot/robotiq_85_gripper/meshes/visual/robotiq_85_knuckle_link.dae"/>
+          <mesh filename="package://costar_simulation/robot/robotiq_85_gripper/meshes/visual/robotiq_85_knuckle_link.dae.obj"/>
         </geometry>
       </visual>
@@ -74,5 +74,5 @@
         <origin rpy="${0.5 * pi} 0 0" xyz="0.0 0.0 0.0"/>
         <geometry>
-          <mesh filename="package://costar_simulation/robot/robotiq_85_gripper/meshes/visual/robotiq_85_knuckle_link.dae"/>
+          <mesh filename="package://costar_simulation/robot/robotiq_85_gripper/meshes/visual/robotiq_85_knuckle_link.dae.obj"/>
         </geometry>
       </visual>
@@ -109,5 +109,5 @@
         <origin rpy="${0.5 * pi} 0 0" xyz="0.0 0.0 0.0"/>
         <geometry>
-          <mesh filename="package://costar_simulation/robot/robotiq_85_gripper/meshes/visual/robotiq_85_finger_link.dae"/>
+          <mesh filename="package://costar_simulation/robot/robotiq_85_gripper/meshes/visual/robotiq_85_finger_link.dae.obj"/>
         </geometry>
       </visual>
@@ -135,5 +135,5 @@
         <origin rpy="${0.5 * pi} 0 0" xyz="0.0 0.0 0.0"/>
         <geometry>
-          <mesh filename="package://costar_simulation/robot/robotiq_85_gripper/meshes/visual/robotiq_85_finger_link.dae"/>
+          <mesh filename="package://costar_simulation/robot/robotiq_85_gripper/meshes/visual/robotiq_85_finger_link.dae.obj"/>
         </geometry>
       </visual>
@@ -177,5 +177,5 @@
         <origin rpy="${0.5 * pi} 0 0" xyz="0.0 0.0 0.0"/>
         <geometry>
-          <mesh filename="package://costar_simulation/robot/robotiq_85_gripper/meshes/visual/robotiq_85_inner_knuckle_link.dae"/>
+          <mesh filename="package://costar_simulation/robot/robotiq_85_gripper/meshes/visual/robotiq_85_inner_knuckle_link.dae.obj"/>
         </geometry>
       </visual>
@@ -203,5 +203,5 @@
         <origin rpy="${0.5 * pi} 0 0" xyz="0.0 0.0 0.0"/>
         <geometry>
-          <mesh filename="package://costar_simulation/robot/robotiq_85_gripper/meshes/visual/robotiq_85_inner_knuckle_link.dae"/>
+          <mesh filename="package://costar_simulation/robot/robotiq_85_gripper/meshes/visual/robotiq_85_inner_knuckle_link.dae.obj"/>
         </geometry>
       </visual>
@@ -240,5 +240,5 @@
         <origin rpy="${0.5 * pi} 0 0" xyz="0.0 0.0 0.0"/>
         <geometry>
-          <mesh filename="package://costar_simulation/robot/robotiq_85_gripper/meshes/visual/robotiq_85_finger_tip_link.dae"/>
+          <mesh filename="package://costar_simulation/robot/robotiq_85_gripper/meshes/visual/robotiq_85_finger_tip_link.dae.obj"/>
         </geometry>
       </visual>
@@ -266,5 +266,5 @@
         <origin rpy="${0.5 * pi} 0 0" xyz="0.0 0.0 0.0"/>
         <geometry>
-          <mesh filename="package://costar_simulation/robot/robotiq_85_gripper/meshes/visual/robotiq_85_finger_tip_link.dae"/>
+          <mesh filename="package://costar_simulation/robot/robotiq_85_gripper/meshes/visual/robotiq_85_finger_tip_link.dae.obj"/>
         </geometry>
       </visual>

Commit message: Merge branch 'feature/sim-updates' of github.com:cpaxton/costar_plan into feature/sim-updates

File: costar_simulation/robot/robotiq_85_gripper/urdf/robotiq_85_gripper.urdf.xacro (robot description, xacro)
@@ -15,7 +15,8 @@
       <visual>
         <material name="blackish"/>
-        <origin rpy="${0.5 * pi} 0 0" xyz="0.0 0.0 0.0"/>
-        <geometry>
-          <mesh filename="package://costar_simulation/robot/robotiq_85_gripper/meshes/visual/robotiq_85_base_link.dae.obj"/>
+        <!--<origin rpy="${0.5 * pi} 0 0" xyz="0.0 0.0 0.0"/>-->
+        <origin xyz="0. 0. 0."/>
+        <geometry>
+          <mesh filename="package://costar_simulation/robot/robotiq_85_gripper/meshes/visual/robotiq_85_base_link.dae"/>
         </geometry>
       </visual>
@@ -51,7 +52,8 @@
       <visual>
         <material name="blackish"/>
-        <origin rpy="${0.5 * pi} 0 0" xyz="0.0 0.0 0.0"/>
-        <geometry>
-          <mesh filename="package://costar_simulation/robot/robotiq_85_gripper/meshes/visual/robotiq_85_knuckle_link.dae.obj"/>
+        <!--<origin rpy="${0.5 * pi} 0 0" xyz="0.0 0.0 0.0"/>-->
+        <origin xyz="0. 0. 0."/>
+        <geometry>
+          <mesh filename="package://costar_simulation/robot/robotiq_85_gripper/meshes/visual/robotiq_85_knuckle_link.dae"/>
         </geometry>
       </visual>
@@ -72,7 +74,8 @@
       <visual>
         <material name="blackish"/>
-        <origin rpy="${0.5 * pi} 0 0" xyz="0.0 0.0 0.0"/>
-        <geometry>
-          <mesh filename="package://costar_simulation/robot/robotiq_85_gripper/meshes/visual/robotiq_85_knuckle_link.dae.obj"/>
+        <!--<origin rpy="${0.5 * pi} 0 0" xyz="0.0 0.0 0.0"/>-->
+        <origin xyz="0. 0. 0."/>
+        <geometry>
+          <mesh filename="package://costar_simulation/robot/robotiq_85_gripper/meshes/visual/robotiq_85_knuckle_link.dae"/>
         </geometry>
       </visual>
@@ -107,7 +110,8 @@
       <visual>
         <material name="blackish"/>
-        <origin rpy="${0.5 * pi} 0 0" xyz="0.0 0.0 0.0"/>
-        <geometry>
-          <mesh filename="package://costar_simulation/robot/robotiq_85_gripper/meshes/visual/robotiq_85_finger_link.dae.obj"/>
+        <!--<origin rpy="${0.5 * pi} 0 0" xyz="0.0 0.0 0.0"/>-->
+        <origin xyz="0. 0. 0."/>
+        <geometry>
+          <mesh filename="package://costar_simulation/robot/robotiq_85_gripper/meshes/visual/robotiq_85_finger_link.dae"/>
         </geometry>
       </visual>
@@ -133,7 +137,8 @@
       <visual>
         <material name="blackish"/>
-        <origin rpy="${0.5 * pi} 0 0" xyz="0.0 0.0 0.0"/>
-        <geometry>
-          <mesh filename="package://costar_simulation/robot/robotiq_85_gripper/meshes/visual/robotiq_85_finger_link.dae.obj"/>
+        <!--<origin rpy="${0.5 * pi} 0 0" xyz="0.0 0.0 0.0"/>-->
+        <origin xyz="0. 0. 0."/>
+        <geometry>
+          <mesh filename="package://costar_simulation/robot/robotiq_85_gripper/meshes/visual/robotiq_85_finger_link.dae"/>
         </geometry>
       </visual>
@@ -175,7 +180,8 @@
       <visual>
         <material name="blackish"/>
-        <origin rpy="${0.5 * pi} 0 0" xyz="0.0 0.0 0.0"/>
-        <geometry>
-          <mesh filename="package://costar_simulation/robot/robotiq_85_gripper/meshes/visual/robotiq_85_inner_knuckle_link.dae.obj"/>
+        <!--<origin rpy="${0.5 * pi} 0 0" xyz="0.0 0.0 0.0"/>-->
+        <origin xyz="0. 0. 0."/>
+        <geometry>
+          <mesh filename="package://costar_simulation/robot/robotiq_85_gripper/meshes/visual/robotiq_85_inner_knuckle_link.dae"/>
         </geometry>
       </visual>
@@ -201,7 +207,8 @@
       <visual>
         <material name="blackish"/>
-        <origin rpy="${0.5 * pi} 0 0" xyz="0.0 0.0 0.0"/>
-        <geometry>
-          <mesh filename="package://costar_simulation/robot/robotiq_85_gripper/meshes/visual/robotiq_85_inner_knuckle_link.dae.obj"/>
+        <!--<origin rpy="${0.5 * pi} 0 0" xyz="0.0 0.0 0.0"/>-->
+        <origin xyz="0. 0. 0."/>
+        <geometry>
+          <mesh filename="package://costar_simulation/robot/robotiq_85_gripper/meshes/visual/robotiq_85_inner_knuckle_link.dae"/>
         </geometry>
       </visual>
@@ -238,7 +245,8 @@
       <visual>
         <material name="blackish"/>
-        <origin rpy="${0.5 * pi} 0 0" xyz="0.0 0.0 0.0"/>
-        <geometry>
-          <mesh filename="package://costar_simulation/robot/robotiq_85_gripper/meshes/visual/robotiq_85_finger_tip_link.dae.obj"/>
+        <!--<origin rpy="${0.5 * pi} 0 0" xyz="0.0 0.0 0.0"/>-->
+        <origin xyz="0. 0. 0."/>
+        <geometry>
+          <mesh filename="package://costar_simulation/robot/robotiq_85_gripper/meshes/visual/robotiq_85_finger_tip_link.dae"/>
         </geometry>
       </visual>
@@ -264,7 +272,8 @@
       <visual>
         <material name="blackish"/>
-        <origin rpy="${0.5 * pi} 0 0" xyz="0.0 0.0 0.0"/>
-        <geometry>
-          <mesh filename="package://costar_simulation/robot/robotiq_85_gripper/meshes/visual/robotiq_85_finger_tip_link.dae.obj"/>
+        <!--<origin rpy="${0.5 * pi} 0 0" xyz="0.0 0.0 0.0"/>-->
+        <origin xyz="0. 0. 0."/>
+        <geometry>
+          <mesh filename="package://costar_simulation/robot/robotiq_85_gripper/meshes/visual/robotiq_85_finger_tip_link.dae"/>
         </geometry>
       </visual>

File: costar_simulation/robot/ur5/ur5.urdf.xacro (robot description, xacro)
@@ -71,7 +71,8 @@
     <link name="${prefix}base_link" >
       <visual>
-        <origin rpy="${0.5 * pi} 0 0" xyz="0.0 0.0 0.0"/>
-        <geometry>
-          <mesh filename="package://costar_simulation/meshes/ur5/visual/Base.dae.obj" />
+        <!--<origin rpy="${0.5 * pi} 0 0" xyz="0.0 0.0 0.0"/>-->
+        <origin xyz="0. 0. 0."/>
+        <geometry>
+          <mesh filename="package://costar_simulation/meshes/ur5/visual/Base.dae" />
         </geometry>
         <material name="LightGrey">
@@ -103,7 +104,8 @@
     <link name="${prefix}shoulder_link">
       <visual>
-        <origin rpy="${0.5 * pi} 0 0" xyz="0.0 0.0 0.0"/>
-        <geometry>
-          <mesh filename="package://costar_simulation/meshes/ur5/visual/Shoulder.dae.obj" />
+        <!--<origin rpy="${0.5 * pi} 0 0" xyz="0.0 0.0 0.0"/>-->
+        <origin xyz="0. 0. 0."/>
+        <geometry>
+          <mesh filename="package://costar_simulation/meshes/ur5/visual/Shoulder.dae" />
         </geometry>
         <material name="LightGrey">
@@ -135,7 +137,8 @@
     <link name="${prefix}upper_arm_link">
       <visual>
-        <origin rpy="${0.5 * pi} 0 0" xyz="0.0 0.0 0.0"/>
-        <geometry>
-          <mesh filename="package://costar_simulation/meshes/ur5/visual/UpperArm.dae.obj" />
+        <!--<origin rpy="${0.5 * pi} 0 0" xyz="0.0 0.0 0.0"/>-->
+        <origin xyz="0. 0. 0."/>
+        <geometry>
+          <mesh filename="package://costar_simulation/meshes/ur5/visual/UpperArm.dae" />
         </geometry>
         <material name="LightGrey">
@@ -167,7 +170,8 @@
     <link name="${prefix}forearm_link">
       <visual>
-        <origin rpy="${0.5 * pi} 0 0" xyz="0.0 0.0 0.0"/>
-        <geometry>
-          <mesh filename="package://costar_simulation/meshes/ur5/visual/Forearm.dae.obj" />
+        <!--<origin rpy="${0.5 * pi} 0 0" xyz="0.0 0.0 0.0"/>-->
+        <origin xyz="0. 0. 0."/>
+        <geometry>
+          <mesh filename="package://costar_simulation/meshes/ur5/visual/Forearm.dae" />
         </geometry>
         <material name="LightGrey">
@@ -199,7 +203,8 @@
     <link name="${prefix}wrist_1_link">
       <visual>
-        <origin rpy="${0.5 * pi} 0 0" xyz="0.0 0.0 0.0"/>
-        <geometry>
-          <mesh filename="package://costar_simulation/meshes/ur5/visual/Wrist1.dae.obj" />
+        <!--<origin rpy="${0.5 * pi} 0 0" xyz="0.0 0.0 0.0"/>-->
+        <origin xyz="0. 0. 0."/>
+        <geometry>
+          <mesh filename="package://costar_simulation/meshes/ur5/visual/Wrist1.dae" />
         </geometry>
         <material name="LightGrey">
@@ -231,7 +236,8 @@
     <link name="${prefix}wrist_2_link">
       <visual>
-        <origin rpy="${0.5 * pi} 0 0" xyz="0.0 0.0 0.0"/>
-        <geometry>
-          <mesh filename="package://costar_simulation/meshes/ur5/visual/Wrist2.dae.obj" />
+        <!--<origin rpy="${0.5 * pi} 0 0" xyz="0.0 0.0 0.0"/>-->
+        <origin xyz="0. 0. 0."/>
+        <geometry>
+          <mesh filename="package://costar_simulation/meshes/ur5/visual/Wrist2.dae" />
         </geometry>
         <material name="LightGrey">
@@ -263,7 +269,8 @@
     <link name="${prefix}wrist_3_link">
       <visual>
-        <origin rpy="${0.5 * pi} 0 0" xyz="0.0 0.0 0.0"/>
-        <geometry>
-          <mesh filename="package://costar_simulation/meshes/ur5/visual/Wrist3.dae.obj" />
+        <!--<origin rpy="${0.5 * pi} 0 0" xyz="0.0 0.0 0.0"/>-->
+        <origin xyz="0. 0. 0."/>
+        <geometry>
+          <mesh filename="package://costar_simulation/meshes/ur5/visual/Wrist3.dae" />
         </geometry>
         <material name="LightGrey">
