Commit message: update xacro

File: costar_simulation/urdf/table/tom_table.urdf.xacro (robot description, xacro)
@@ -1,4 +1,4 @@
 <?xml version="0.0" ?>
-<robot name="table.urdf">
+<robot xmlns:xacro="http://www.ros.org/wiki/xacro">
   <xacro:macro name="top_panel">
     <geometry>
@@ -25,21 +25,31 @@
     <color rgba="0.8 0.8 0.8 1."/>
   </material>
-  <link name="baseLink">
-    <contact>
-      <lateral_friction value="1.0"/>
-    </contact>
-    <inertial>
-      <origin rpy="0 0 0" xyz="0 0 0"/>
-      <mass value=".0"/>
-      <inertia ixx="1" ixy="0" ixz="0" iyy="1" iyz="0" izz="1"/>
-    </inertial>
-    <visual>
-      <origin rpy="0 0 0" xyz="0 0.3 -0.0085"/>
-      <xacro:top_panel/>
-    </visual>
-    <visual>
-      <origin rpy="0 0 0" xyz="0 0.3 -0.00285"/>
-      <xacro:top_base/>
-    </visual>
-  </link>
+  <xacro:macro name="tom_table" params="name">
+    <link name="${name}">
+      <contact>
+        <lateral_friction value="1.0"/>
+      </contact>
+      <inertial>
+        <origin rpy="0 0 0" xyz="0 0 0"/>
+        <mass value=".0"/>
+        <inertia ixx="1" ixy="0" ixz="0" iyy="1" iyz="0" izz="1"/>
+      </inertial>
+      <visual>
+        <origin rpy="0 0 0" xyz="0 0.3 -0.0085"/>
+        <xacro:top_panel/>
+      </visual>
+      <collision>
+        <origin rpy="0 0 0" xyz="0 0.3 -0.0085"/>
+        <xacro:top_panel/>
+      </collision>
+      <visual>
+        <origin rpy="0 0 0" xyz="0 0.3 -0.00285"/>
+        <xacro:top_base/>
+      </visual>
+      <collision>
+        <origin rpy="0 0 0" xyz="0 0.3 -0.00285"/>
+        <xacro:top_base/>
+      </collision>
+    </link>
+  </xacro:macro>
 </robot>
