Commit message: update table model

File: costar_simulation/urdf/table/tom_table.xacro (robot description, xacro)
@@ -3,5 +3,5 @@
   <xacro:macro name="top_panel">
     <geometry>
-      <box size="1 0.6 0.017"/>
+      <box size="1 0.595 0.017"/>
     </geometry>
     <material name="dark"/>
@@ -9,5 +9,5 @@
   <xacro:macro name="top_base">
     <geometry>
-      <box size="1 0.6 0.04"/>
+      <box size="1 0.595 0.04"/>
     </geometry>
     <material name="light"/>
@@ -18,4 +18,14 @@
     </geometry>
     <material name="light"/>
+  </xacro:macro>
+  <xacro:macro name="leg_at" params="xyz">
+    <visual>
+      <origin rpy="0 0 0" xyz="${xyz}"/>
+      <xacro:leg/>
+    </visual>
+    <collision>
+      <origin rpy="0 0 0" xyz="${xyz}"/>
+      <xacro:leg/>
+    </collision>
   </xacro:macro>
   <material name="dark">
@@ -36,19 +46,23 @@
       </inertial>
       <visual>
-        <origin rpy="0 0 0" xyz="0 0.3 -0.0085"/>
+        <origin rpy="0 0 0" xyz="0 ${0.595 / 2} -0.0085"/>
         <xacro:top_panel/>
       </visual>
       <collision>
-        <origin rpy="0 0 0" xyz="0 0.3 -0.0085"/>
+        <origin rpy="0 0 0" xyz="0 ${0.595 / 2} -0.0085"/>
         <xacro:top_panel/>
       </collision>
       <visual>
-        <origin rpy="0 0 0" xyz="0 0.3 -0.00285"/>
+        <origin rpy="0 0 0" xyz="0 ${0.595 / 2} -0.00285"/>
         <xacro:top_base/>
       </visual>
       <collision>
-        <origin rpy="0 0 0" xyz="0 0.3 -0.00285"/>
+        <origin rpy="0 0 0" xyz="0 ${0.595 / 2} -0.00285"/>
         <xacro:top_base/>
       </collision>
+      <xacro:leg_at xyz="-0.5 0.02 ${-0.00285 + (0.823 / 2)}"/>
+      <xacro:leg_at xyz="0.5 0.02 ${-0.00285 + (0.823 / 2)}"/>
+      <xacro:leg_at xyz="-0.5 ${0.595 - 0.02} ${-0.00285 + (0.823 / 2)}"/>
+      <xacro:leg_at xyz="0.5 ${0.595 - 0.02} ${-0.00285 + (0.823 / 2)}"/>
     </link>
   </xacro:macro>

Commit message: updates

File: costar_simulation/urdf/table/tom_table.xacro (robot description, xacro)
@@ -1,4 +1,11 @@
 <?xml version="0.0" ?>
 <robot xmlns:xacro="http://www.ros.org/wiki/xacro">
+  <xacro:property name="M_PI" value="3.14159"/>
+  <material name="dark">
+    <color rgba="0.3 0.3 0.3 1."/>
+  </material>
+  <material name="light">
+    <color rgba="0.3 0.3 0.3 1."/>
+  </material>
   <xacro:macro name="top_panel">
     <geometry>
@@ -29,10 +36,4 @@
     </collision>
   </xacro:macro>
-  <material name="dark">
-    <color rgba="0.2 0.2 0.2 1."/>
-  </material>
-  <material name="light">
-    <color rgba="0.8 0.8 0.8 1."/>
-  </material>
   <xacro:macro name="tom_table" params="name">
     <link name="${name}">
@@ -54,15 +55,15 @@
       </collision>
       <visual>
-        <origin rpy="0 0 0" xyz="0 ${0.595 / 2} -0.00285"/>
+        <origin rpy="0 0 0" xyz="0 ${0.595 / 2} ${-0.017 - 0.02}"/>
         <xacro:top_base/>
       </visual>
       <collision>
-        <origin rpy="0 0 0" xyz="0 ${0.595 / 2} -0.00285"/>
+        <origin rpy="0 0 0" xyz="0 ${0.595 / 2} ${-0.017 - 0.02}"/>
         <xacro:top_base/>
       </collision>
-      <xacro:leg_at xyz="-0.5 0.02 ${-0.00285 + (0.823 / 2)}"/>
-      <xacro:leg_at xyz="0.5 0.02 ${-0.00285 + (0.823 / 2)}"/>
-      <xacro:leg_at xyz="-0.5 ${0.595 - 0.02} ${-0.00285 + (0.823 / 2)}"/>
-      <xacro:leg_at xyz="0.5 ${0.595 - 0.02} ${-0.00285 + (0.823 / 2)}"/>
+      <xacro:leg_at xyz="${-0.5+0.02} 0.02 ${-0.017 - 0.02 - (0.823 / 2)}"/>
+      <xacro:leg_at xyz="${0.5-0.02} 0.02 ${-0.017 -0.02 - (0.823 / 2)}"/>
+      <xacro:leg_at xyz="${-0.5+0.02} ${0.595 - 0.02} ${-0.017 - 0.02 - (0.823 / 2)}"/>
+      <xacro:leg_at xyz="${0.5-0.02} ${0.595 - 0.02} ${-0.017 -0.02 - (0.823 / 2)}"/>
     </link>
   </xacro:macro>

Commit message: making a bunch of changes to set up the table at a particular position

File: costar_simulation/urdf/table/tom_table.xacro (robot description, xacro)
@@ -2,21 +2,15 @@
 <robot xmlns:xacro="http://www.ros.org/wiki/xacro">
   <xacro:property name="M_PI" value="3.14159"/>
-  <material name="dark">
-    <color rgba="0.3 0.3 0.3 1."/>
+  <material name="tt_metal">
+    <color rgba="0.75 0.75 0.75 1."/>
   </material>
-  <material name="light">
-    <color rgba="0.3 0.3 0.3 1."/>
+  <material name="tt_top">
+    <color rgba="0.2 0.2 0.2 1."/>
   </material>
-  <xacro:macro name="top_panel">
-    <geometry>
-      <box size="1 0.595 0.017"/>
-    </geometry>
-    <material name="dark"/>
-  </xacro:macro>
   <xacro:macro name="top_base">
     <geometry>
       <box size="1 0.595 0.04"/>
     </geometry>
-    <material name="light"/>
+    <material name="tt_metal"/>
   </xacro:macro>
   <xacro:macro name="leg">
@@ -24,5 +18,5 @@
       <box size="0.04 0.04 0.823"/>
     </geometry>
-    <material name="light"/>
+    <material name="tt_metal"/>
   </xacro:macro>
   <xacro:macro name="leg_at" params="xyz">
@@ -35,4 +29,10 @@
       <xacro:leg/>
     </collision>
+  </xacro:macro>
+  <xacro:macro name="top_panel">
+    <geometry>
+      <box size="1 0.595 0.017"/>
+    </geometry>
+    <material name="tt_metal"/>
   </xacro:macro>
   <xacro:macro name="tom_table" params="name">
