Commit message: updating poses

File: costar_simulation/urdf/duplo/duplo.xacro (robot description, xacro)
@@ -12,5 +12,5 @@
         <origin rpy="0 0 0" xyz="0 0 0"/>
         <geometry>
-          <box size="0.127 0.087 0.063"/>
+          <box size="0.127 0.063 0.087"/>
         </geometry>
       </collision>
