Commit message: mesh and geometry

File: costar_simulation/urdf/box/box.urdf.xacro (robot description, xacro)
@@ -1,5 +1,5 @@
 <?xml version="0.0" ?>
-<robot name="block_1" xmlns:xacro="http://www.ros.org/wiki/xacro">
-  <xacro:include filename="$(find costar_simulation)/urdf/duplo/duplo.xacro"/>
-  <xacro:duplo name="block_1"/>
+<robot name="box" xmlns:xacro="http://www.ros.org/wiki/xacro">
+  <xacro:include filename="$(find costar_simulation)/urdf/box/box.xacro"/>
+  <xacro:box name="box"/>
 </robot>

File: costar_simulation/urdf/box/box.xacro (robot description, xacro)
@@ -1,10 +1,10 @@
 <?xml version="0.0" ?>
 <robot xmlns:xacro="http://www.ros.org/wiki/xacro">
-  <xacro:macro name="duplo" params="name">
+  <xacro:macro name="box" params="name">
     <link name="${name}">
       <visual>
         <origin rpy="0 0 0" xyz="0 0 0"/>
         <geometry>
-          <mesh filename="package://costar_simulation/urdf/duplo/duplo.dae" scale="1. 1. 1."/>
+          <mesh filename="package://costar_simulation/urdf/box/box.dae" scale="1. 1. 1."/>
         </geometry>
       </visual>
@@ -12,5 +12,5 @@
         <origin rpy="0 0 0" xyz="0 0 0"/>
         <geometry>
-          <box size="0.127 0.063 0.087"/>
+          <box size="0.205 0.205 0.205"/>
         </geometry>
       </collision>

Commit message: update scene: display the box in the correct place

File: costar_simulation/urdf/box/box.urdf.xacro (robot description, xacro)
@@ -1,5 +1,6 @@
 <?xml version="0.0" ?>
 <robot name="box" xmlns:xacro="http://www.ros.org/wiki/xacro">
-  <xacro:include filename="$(find costar_simulation)/urdf/box/box.xacro"/>
-  <xacro:box name="box"/>
+  <xacro:include
+    filename="$(find costar_simulation)/urdf/box/box.xacro"/>
+  <xacro:tom_box name="box"/>
 </robot>

File: costar_simulation/urdf/box/box.xacro (robot description, xacro)
@@ -1,5 +1,6 @@
 <?xml version="0.0" ?>
 <robot xmlns:xacro="http://www.ros.org/wiki/xacro">
-  <xacro:macro name="box" params="name">
+  <xacro:macro name="tom_box" params="name">
+    <xacro:property name="M_PI" value="3.14159"/>
     <link name="${name}">
       <visual>
