Commit message: tweak drill model definitions

File: costar_simulation/urdf/drill/drill.xacro (robot description, xacro)
@@ -2,4 +2,7 @@
 <robot xmlns:xacro="http://www.ros.org/wiki/xacro">
   <xacro:macro name="drill" params="name">
+    <material name="darkblue">
+      <color rgba="0.2 0.2 0.4 1"/>
+    </material>
     <link name="${name}">
       <contact>
@@ -20,4 +23,5 @@
       <visual>
         <origin rpy="0 0 0" xyz="0 0 0"/>
+        <material name="darkblue"/>
         <geometry>
           <mesh filename="package://costar_simulation/urdf/drill/drill.stl" scale="1 1 1"/>

File: costar_simulation/urdf/drill/drill_receptacle.xacro (robot description, xacro)
@@ -2,4 +2,7 @@
 <robot xmlns:xacro="http://www.ros.org/wiki/xacro">
   <xacro:macro name="drill_receptacle" params="name">
+    <material name="offwhite">
+      <color rgba="0.9 0.9 0.7 1"/>
+    </material>
     <link name="${name}">
       <contact>
@@ -15,5 +18,5 @@
         <origin rpy="0 0 0" xyz="0 0 0"/>
         <geometry>
-          <mesh filename="package://costar_simulation/urdf/drill/drill_receptacle.dae" scale="1 1 1"/>
+          <mesh filename="package://costar_simulation/urdf/drill/drill_receptacle.stl" scale="1 1 1"/>
         </geometry>
       </collision>
@@ -23,4 +26,5 @@
           <mesh filename="package://costar_simulation/urdf/drill/drill)drill_receptacle.stl" scale="1 1 1"/>
         </geometry>
+        <material name="offwhite"/>
       </visual>
     </link>
