Commit message: add drill objects

File: costar_simulation/urdf/drill/drill_receptacle.xacro (robot description, xacro)
@@ -1,5 +1,5 @@
 <?xml version="0.0" ?>
 <robot xmlns:xacro="http://www.ros.org/wiki/xacro">
-  <xacro:macro name="drill" params="name">
+  <xacro:macro name="drill_receptacle" params="name">
     <link name="${name}">
       <contact>
@@ -15,5 +15,5 @@
         <origin rpy="0 0 0" xyz="0 0 0"/>
         <geometry>
-          <mesh filename="package://costar_simulation/urdf/drill/drill.dae" scale="1 1 1"/>
+          <mesh filename="package://costar_simulation/urdf/drill/drill_receptacle.dae" scale="1 1 1"/>
         </geometry>
       </collision>
@@ -21,5 +21,5 @@
         <origin rpy="0 0 0" xyz="0 0 0"/>
         <geometry>
-          <mesh filename="package://costar_simulation/urdf/drill/drill.stl" scale="1 1 1"/>
+          <mesh filename="package://costar_simulation/urdf/drill/drill)drill_receptacle.stl" scale="1 1 1"/>
         </geometry>
       </visual>

Commit message: fix various bugs

File: costar_simulation/urdf/drill/drill_receptacle.xacro (robot description, xacro)
@@ -24,5 +24,5 @@
         <origin rpy="0 0 0" xyz="0 0 0"/>
         <geometry>
-          <mesh filename="package://costar_simulation/urdf/drill/drill)drill_receptacle.stl" scale="1 1 1"/>
+          <mesh filename="package://costar_simulation/urdf/drill/drill_receptacle.stl" scale="1 1 1"/>
         </geometry>
         <material name="offwhite"/>
